Commit message: Update gazebo camera model to include RGBD sensor

File: description/zed_camera.xacro (robot description, xacro)
@@ -28,7 +28,8 @@
     <link name="${prefix}zedm_left_camera_frame" />
     <joint name="${prefix}zedm_left_camera_optical_joint" type="fixed">
-        <origin xyz="0 0 0" rpy="-1.57079632679 0.0 -1.57079632679"/>
         <parent link="${prefix}zedm_left_camera_frame"/>
         <child link="${prefix}zedm_left_camera_optical_frame"/>
+        <!-- <origin xyz="0 0 0" rpy="-1.57079632679 0.0 -1.57079632679"/> -->
+        <origin xyz="0 0 0" rpy="0 0 0"/>
     </joint>
     <link name="${prefix}zedm_left_camera_optical_frame"/>
@@ -41,19 +42,40 @@
     <link name="${prefix}zedm_right_camera_frame" />
     <joint name="${prefix}zedm_right_camera_optical_joint" type="fixed">
-        <origin xyz="0 0 0" rpy="-1.57079632679 0.0 -1.57079632679"/>
         <parent link="${prefix}zedm_right_camera_frame"/>
         <child link="${prefix}zedm_right_camera_optical_frame"/>
+        <origin xyz="0 0 0" rpy="-1.57079632679 0.0 -1.57079632679"/>
     </joint>
     <link name="${prefix}zedm_right_camera_optical_frame"/>
-    <!-- <gazebo reference="${prefix}zedm_camera_center">
-        <material>Gazebo/Green</material>
-    </gazebo> -->
+    <!-- Left Camera Gazebo -->
     <gazebo reference="${prefix}zedm_left_camera_frame">
-        <sensor name="${prefix}left_camera" type="camera">
-            <pose> 0 0 0 0 0 0 </pose>
+        <sensor name="${prefix}left_camera" type="rgbd_camera">
+          <topic>camera/left_camera</topic>
+          <gz_frame_id>zedm_left_camera_optical_frame</gz_frame_id>
+          <always_on>1</always_on>
+          <update_rate>10</update_rate>
+          <visualize>true</visualize>
+          <camera>
+            <horizontal_fov>1.089</horizontal_fov>
+            <image>
+              <width>640</width>
+              <height>480</height>
+              <format>R_FLOAT32</format>
+            </image>
+            <clip>
+              <near>0.1</near>
+              <far>100</far>
+            </clip>
+          </camera>
+        </sensor>
+    </gazebo>
+    <!-- Right Camera Gazebo -->
+    <gazebo reference="${prefix}zedm_right_camera_frame">
+        <sensor name="${prefix}right_camera" type="camera">
+            <topic>camera/right_camera/image</topic>
+            <gz_frame_id>zedm_right_camera_optical_frame</gz_frame_id>
             <visualize>true</visualize>
             <update_rate>30</update_rate>
             <camera>
-                <camera_info_topic>camera/left_camera_info</camera_info_topic>
+                <camera_info_topic>camera/right_camera/camera_info</camera_info_topic>
                 <horizontal_fov>1.089</horizontal_fov>
                 <image>
@@ -67,28 +89,4 @@
                 </clip>
             </camera>
-            <topic>camera/left_camera_image_raw</topic>
-            <gz_frame_id>zedm_left_camera_optical_frame</gz_frame_id>
-        </sensor>
-    </gazebo>
-    <gazebo reference="${prefix}zedm_right_camera_frame">
-        <sensor name="${prefix}right_camera" type="camera">
-            <pose> 0 0 0 0 0 0 </pose>
-            <visualize>true</visualize>
-            <update_rate>30</update_rate>
-            <camera>
-                <camera_info_topic>camera/right_camera_info</camera_info_topic>
-                <horizontal_fov>1.089</horizontal_fov>
-                <image>
-                    <format>R8G8B8</format>
-                    <width>640</width>
-                    <height>480</height>
-                </image>
-                <clip>
-                    <near>0.05</near>
-                    <far>8.0</far>
-                </clip>
-            </camera>
-            <topic>camera/right_camera_image_raw</topic>
-            <gz_frame_id>zedm_right_camera_optical_frame</gz_frame_id>
         </sensor>
     </gazebo>
