Commit message: refactored robot description code

File: description/robot_core.xacro (robot description, xacro)
@@ -25,5 +25,5 @@
         filename="package://cohort/meshes/base_link.STL" /> -->
         <mesh
-        filename="file://$(find cohort)/meshes/base_link.STL"/>
+        filename="file://$(find arcs_cohort_description)/meshes/new_base_link.stl"/>
     </geometry>
     <material
@@ -39,5 +39,5 @@
     <geometry>
       <mesh
-        filename="file://$(find cohort)/meshes/base_link.STL" />
+        filename="file://$(find arcs_cohort_description)/meshes/new_base_link.stl" />
     </geometry>
   </collision>
@@ -65,5 +65,5 @@
     <geometry>
       <mesh
-        filename="file://$(find cohort)/meshes/front_left_wheel_link.STL" />
+        filename="file://$(find arcs_cohort_description)/meshes/new_front_left_wheel.stl" />
     </geometry>
     <material
@@ -79,5 +79,5 @@
     <geometry>
       <mesh
-        filename="file://$(find cohort)/meshes/front_left_wheel_link.STL" />
+        filename="file://$(find arcs_cohort_description)/meshes/new_front_left_wheel.stl" />
     </geometry>
   </collision>
@@ -118,5 +118,5 @@
     <geometry>
       <mesh
-        filename="file://$(find cohort)/meshes/front_right_wheel_link.STL" />
+        filename="file://$(find arcs_cohort_description)/meshes/new_front_right_wheel.stl" />
     </geometry>
     <material
@@ -132,5 +132,5 @@
     <geometry>
       <mesh
-        filename="file://$(find cohort)/meshes/front_right_wheel_link.STL" />
+        filename="file://$(find arcs_cohort_description)/meshes/new_front_right_wheel.stl" />
     </geometry>
   </collision>
@@ -171,5 +171,5 @@
     <geometry>
       <mesh
-        filename="file://$(find cohort)/meshes/back_left_wheel_link.STL" />
+        filename="file://$(find arcs_cohort_description)/meshes/new_back_left_wheel.stl" />
     </geometry>
     <material
@@ -185,5 +185,5 @@
     <geometry>
       <mesh
-        filename="file://$(find cohort)/meshes/back_left_wheel_link.STL" />
+        filename="file://$(find arcs_cohort_description)/meshes/new_back_left_wheel.stl" />
     </geometry>
   </collision>
@@ -224,5 +224,5 @@
     <geometry>
       <mesh
-        filename="file://$(find cohort)/meshes/back_right_wheel_link.STL" />
+        filename="file://$(find arcs_cohort_description)/meshes/new_back_right_wheel.stl" />
     </geometry>
     <material
@@ -238,5 +238,5 @@
     <geometry>
       <mesh
-        filename="file://$(find cohort)/meshes/back_right_wheel_link.STL" />
+        filename="file://$(find arcs_cohort_description)/meshes/new_back_right_wheel.stl" />
     </geometry>
   </collision>
@@ -277,5 +277,5 @@
     <geometry>
       <mesh
-        filename="file://$(find cohort)/meshes/imu_link.STL" />
+        filename="file://$(find arcs_cohort_description)/meshes/new_imu.stl" />
     </geometry>
     <material
@@ -291,5 +291,5 @@
     <geometry>
       <mesh
-        filename="file://$(find cohort)/meshes/imu_link.STL" />
+        filename="file://$(find arcs_cohort_description)/meshes/new_imu.stl" />
     </geometry>
   </collision>
@@ -330,5 +330,5 @@
     <geometry>
       <mesh
-        filename="file://$(find cohort)/meshes/camera_mount_link.STL" />
+        filename="file://$(find arcs_cohort_description)/meshes/new_camera_mount.stl" />
     </geometry>
     <material
@@ -344,5 +344,5 @@
     <geometry>
       <mesh
-        filename="file://$(find cohort)/meshes/camera_mount_link.STL" />
+        filename="file://$(find arcs_cohort_description)/meshes/new_camera_mount.stl" />
     </geometry>
   </collision>
@@ -383,5 +383,5 @@
     <geometry>
       <mesh
-        filename="file://$(find cohort)/meshes/zedmini_center_link.STL" />
+        filename="file://$(find arcs_cohort_description)/meshes/zedmini_center_link.STL" />
     </geometry>
     <material
@@ -397,5 +397,5 @@
     <geometry>
       <mesh
-        filename="file://$(find cohort)/meshes/zedmini_center_link.STL" />
+        filename="file://$(find arcs_cohort_description)/meshes/zedmini_center_link.STL" />
     </geometry>
   </collision>

File: description/zed_camera.xacro (robot description, xacro)
@@ -12,5 +12,5 @@
             <geometry>
             <!-- add zed camera stl -->
-                <mesh filename="file://$(find cohort)/meshes/zedm.stl"/>
+                <mesh filename="file://$(find arcs_cohort_description)/meshes/zedm.stl"/>
             </geometry>
             <material name="black">

Commit message: made changes to the camera description

File: description/robot_core.xacro (robot description, xacro)
@@ -1,4 +1,16 @@
 <?xml version="1.0"?>
 <robot xmlns:xacro="http://www.ros.org/wiki/xacro">
+  <material name="yellow">
+      <color rgba="1 1 0 1"/>
+  </material>
+  <material name="orange">
+      <color rgba="1 0.3 0.1 1"/>
+  </material>
+  <material name="blue">
+      <color rgba="0.2 0.2 1 1"/>
+  </material>
+  <material name="red">
+      <color rgba="1 0 0 1"/>
+  </material>
   <link
   name="base_link">
@@ -17,19 +29,13 @@
       izz="0.00438426362438441" />
   </inertial>
-  <visual>w
-    <origin
-      xyz="0 0 0"
-      rpy="0 0 0" />
-    <geometry>
-      <!-- <mesh
-        filename="package://cohort/meshes/base_link.STL" /> -->
+  <visual>
+    <origin
+      xyz="0 0 0"
+      rpy="0 0 0" />
+    <geometry>
         <mesh
         filename="file://$(find arcs_cohort_description)/meshes/new_base_link.stl"/>
     </geometry>
-    <material
-      name="">
-      <color
-        rgba="0.752941176470588 0.752941176470588 0.752941176470588 1" />
-    </material>
+    <material name="blue"/>
   </visual>
   <collision>
@@ -67,9 +73,5 @@
         filename="file://$(find arcs_cohort_description)/meshes/new_front_left_wheel.stl" />
     </geometry>
-    <material
-      name="">
-      <color
-        rgba="1 1 1 1" />
-    </material>
+    <material name="orange"/>
   </visual>
   <collision>
@@ -120,9 +122,5 @@
         filename="file://$(find arcs_cohort_description)/meshes/new_front_right_wheel.stl" />
     </geometry>
-    <material
-      name="">
-      <color
-        rgba="1 1 1 1" />
-    </material>
+    <material name="orange"/>
   </visual>
   <collision>
@@ -173,9 +171,5 @@
         filename="file://$(find arcs_cohort_description)/meshes/new_back_left_wheel.stl" />
     </geometry>
-    <material
-      name="">
-      <color
-        rgba="1 1 1 1" />
-    </material>
+    <material name="orange"/>
   </visual>
   <collision>
@@ -226,9 +220,5 @@
         filename="file://$(find arcs_cohort_description)/meshes/new_back_right_wheel.stl" />
     </geometry>
-    <material
-      name="">
-      <color
-        rgba="1 1 1 1" />
-    </material>
+    <material name="orange"/>
   </visual>
   <collision>
@@ -332,9 +322,5 @@
         filename="file://$(find arcs_cohort_description)/meshes/new_camera_mount.stl" />
     </geometry>
-    <material
-      name="">
-      <color
-        rgba="1 1 1 1" />
-    </material>
+    <material name="red"/>
   </visual>
   <collision>
@@ -386,8 +372,5 @@
     </geometry>
     <material
-      name="">
-      <color
-        rgba="0.792156862745098 0.819607843137255 0.933333333333333 1" />
-    </material>
+      name="yellow"/>
   </visual>
   <collision>

File: description/zed_camera.xacro (robot description, xacro)
@@ -54,4 +54,5 @@
             <update_rate>10</update_rate>
             <camera>
+                <camera_info_topic>camera/left_camera_info</camera_info_topic>
                 <horizontal_fov>1.089</horizontal_fov>
                 <image>
@@ -65,7 +66,9 @@
                 </clip>
             </camera>
-            <plugin name="left_camera_controller" filename="libgazebo_ros_camera.so">
+            <topic>camera/left_camera_image_raw</topic>
+            <gz_frame_id>camera_left_link_optical</gz_frame_id>
+            <!-- <plugin name="left_camera_controller" filename="libgazebo_ros_camera.so">
                 <frame_name>zedm_left_optical_frame</frame_name>
-            </plugin>
+            </plugin> -->
         </sensor>
     </gazebo>
@@ -76,4 +79,5 @@
             <update_rate>10</update_rate>
             <camera>
+                <camera_info_topic>camera/right_camera_info</camera_info_topic>
                 <horizontal_fov>1.089</horizontal_fov>
                 <image>
@@ -87,7 +91,9 @@
                 </clip>
             </camera>
-            <plugin name="right_camera_controller" filename="libgazebo_ros_camera.so">
+            <topic>camera/right_camera_image_raw</topic>
+            <gz_frame_id>camera_right_link_optical</gz_frame_id>
+            <!-- <plugin name="right_camera_controller" filename="libgazebo_ros_camera.so">
                 <frame_name>zedm_right_optical_frame</frame_name>
-            </plugin>
+            </plugin> -->
         </sensor>
     </gazebo>

Commit message: Updated transforms for camera links in robot xacro to match model rotation to transform rotation

File: description/robot_core.xacro (robot description, xacro)
@@ -1,4 +1,5 @@
 <?xml version="1.0"?>
 <robot xmlns:xacro="http://www.ros.org/wiki/xacro">
+  <xacro:property name="M_PI"         value="3.1415926535897931" />
   <!-- Define a macro with a prefix param for the robot description -->
   <xacro:macro name="robot_description" params="prefix">
@@ -283,5 +284,5 @@
         <origin
           xyz="0 0 0"
-          rpy="0 0 0" />
+          rpy="0 -${M_PI/4} 0" />
         <geometry>
           <mesh
@@ -302,5 +303,5 @@
     </link>
     <joint name="${prefix}camera_mount_joint" type="fixed">
-      <origin xyz="0.14426 0.00028171 0.094535" rpy="0 0 0" />
+      <origin xyz="0.14426 0.00028171 0.094535" rpy="0 ${M_PI/4} 0" />
       <parent link="${prefix}base_link" />
       <child link="${prefix}camera_mount_link" />
@@ -309,5 +310,6 @@
     <link name="${prefix}zedmini_center_link">
       <inertial>
-        <origin xyz="-0.00435147007919079 -0.00309486253694627 0.00251127017920943" rpy="0 0 0" />
+      <!-- What are these magic numbers? -->
+        <origin xyz="-0.00435147007919079 -0.00309486253694627 0.00" rpy="0 0 0" />
         <mass value="0.0560548842495178" />
         <inertia
@@ -321,6 +323,6 @@
       <visual>
         <origin
-          xyz="0 0 0"
-          rpy="0 0 0" />
+          xyz="0 0 0.05"
+          rpy="0 -${M_PI/4} 0" />
         <geometry>
           <mesh
@@ -332,5 +334,5 @@
       <collision>
         <origin
-          xyz="0 0 0"
+          xyz="0 0 0.05"
           rpy="0 0 0" />
         <geometry>

File: description/zed_camera.xacro (robot description, xacro)
@@ -54,5 +54,6 @@
     <link name="${prefix}zedm_left_camera_frame" />
     <joint name="${prefix}zedm_left_camera_optical_joint" type="fixed">
-        <origin xyz="0 0 0" rpy="-1.57079632679 0.0 -1.57079632679"/>
+        <!-- <origin xyz="0 0 0" rpy="-1.57079632679 0.0 -1.57079632679"/> -->
+        <origin xyz="0 0 0" rpy="0.0 0.0 0.0"/>
         <parent link="${prefix}zedm_left_camera_frame"/>
         <child link="${prefix}zedm_left_camera_optical_frame"/>

Commit message: Add camera name to additional camera links/joints

File: description/robot_core.xacro (robot description, xacro)
@@ -265,5 +265,5 @@
       <axis xyz="0 0 0" />
     </joint>
-    <link name="${prefix}camera_mount_link">
+    <link name="${prefix}${camera_name}_camera_mount_link">
       <inertial>
         <origin
@@ -304,5 +304,5 @@
       <origin xyz="0.14426 0.00028171 0.094535" rpy="0 0 0" />
       <parent link="${prefix}base_link" />
-      <child link="${prefix}camera_mount_link" />
+      <child link="${prefix}${camera_name}_camera_mount_link" />
       <axis xyz="0 0 0" />
     </joint>
@@ -325,5 +325,5 @@
         <geometry>
           <mesh
-            filename="file://$(find arcs_cohort_description)/meshes/${camera_model}_center_link.STL" />
+            filename="file://$(find arcs_cohort_description)/meshes/${camera_model}_center_link.stl" />
         </geometry>
         <material
@@ -336,5 +336,5 @@
         <geometry>
           <mesh
-            filename="file://$(find arcs_cohort_description)/meshes/${camera_model}_center_link.STL" />
+            filename="file://$(find arcs_cohort_description)/meshes/${camera_model}_center_link.stl" />
           <!-- <box size="0.015 0.122 0.025"/> -->
         </geometry>
@@ -343,5 +343,5 @@
     <joint name="${prefix}${camera_name}_center_joint" type="fixed">
       <origin xyz="0.050151 0.0018215 -0.015053" rpy="0 0 0" />
-      <parent link="${prefix}camera_mount_link" />
+      <parent link="${prefix}${camera_name}_camera_mount_link" />
       <child link="${prefix}${camera_name}_center_link" />
       <axis xyz="0 0 0" />

File: description/zed_camera.xacro (robot description, xacro)
@@ -10,20 +10,20 @@
   <xacro:macro name="zed_camera_description" params="prefix camera_name=zedm camera_model=zedm resolution=VGA">
     <!--Camera-->
-    <!-- <joint name="${prefix}zedm_camera_center_joint" type="fixed">
-        <parent link="${prefix}zedmini_center_link"/>
-        <child link="${prefix}zedm_camera_center"/>
-        <origin xyz="0.305 0 0.08" rpy="0 0 0" />
-    </joint>
-    <link name="${prefix}zedm_camera_center">
-        <visual>
-            <origin xyz="0 0 0" rpy="0 0 0"/>
-            <geometry>
-                <mesh filename="file://$(find arcs_cohort_description)/meshes/zedm.stl"/>
-            </geometry>
-            <material name="black">
-                <color rgba="0 0 0 0.9"/>
-            </material>
-        </visual>
-    </link> -->
+    <!-- <joint name="${prefix}${camera_name}_camera_center_joint" type="fixed"> -->
+    <!--     <parent link="${prefix}${camera_name}_camera_mount_link"/> -->
+    <!--     <child link="${prefix}${camera_name}_camera_center"/> -->
+    <!--     <origin xyz="0.305 0 0.08" rpy="0 0 0" /> -->
+    <!-- </joint> -->
+    <!-- <link name="${prefix}${camera_name}_camera_center"> -->
+    <!--     <visual> -->
+    <!--         <origin xyz="0 0 0" rpy="0 0 0"/> -->
+    <!--         <geometry> -->
+    <!--             <mesh filename="file://$(find arcs_cohort_description)/meshes/zedm.stl"/> -->
+    <!--         </geometry> -->
+    <!--         <material name="black"> -->
+    <!--             <color rgba="0 0 0 0.9"/> -->
+    <!--         </material> -->
+    <!--     </visual> -->
+    <!-- </link> -->
     <xacro:if value="${resolution == 'HD2K'}">
         <xacro:property name="resolution_width" value="2208" />
