Commit message: Modify robot model to use zed_wrapper camera urdf

File: description/robot_core.xacro (robot description, xacro)
@@ -307,44 +307,4 @@
       <axis xyz="0 0 0" />
     </joint>
-    <link name="${prefix}${camera_name}_center_link">
-      <inertial>
-        <origin xyz="-0.00435147007919079 -0.00309486253694627 0.00251127017920943" rpy="0 0 0" />
-        <mass value="0.0560548842495178" />
-        <inertia
-          ixx="7.29762807495571E-05"
-          ixy="5.57132554461124E-07"
-          ixz="-2.34695280152666E-07"
-          iyy="5.49793925654236E-06"
-          iyz="-3.21584411064254E-07"
-          izz="7.2705806093778E-05" />
-      </inertial>
-      <visual>
-        <origin
-          xyz="0 0 0"
-          rpy="0 0 0" />
-        <geometry>
-          <mesh
-            filename="file://$(find arcs_cohort_description)/meshes/${camera_model}_center_link.stl" />
-        </geometry>
-        <material
-          name="yellow"/>
-      </visual>
-      <collision>
-        <origin
-          xyz="0 0 0"
-          rpy="0 0 0" />
-        <geometry>
-          <mesh
-            filename="file://$(find arcs_cohort_description)/meshes/${camera_model}_center_link.stl" />
-          <!-- <box size="0.015 0.122 0.025"/> -->
-        </geometry>
-      </collision>
-    </link>
-    <joint name="${prefix}${camera_name}_center_joint" type="fixed">
-      <origin xyz="0.050151 0.0018215 -0.015053" rpy="0 0 0" />
-      <parent link="${prefix}${camera_name}_camera_mount_link" />
-      <child link="${prefix}${camera_name}_center_link" />
-      <axis xyz="0 0 0" />
-    </joint>
   </xacro:macro>
 </robot>

File: description/zed_camera.xacro (robot description, xacro)
@@ -7,150 +7,122 @@
 -->
 <robot xmlns:xacro="http://www.ros.org/wiki/xacro" >
-  <!-- Define a macro with a prefix param for the Zed M camera description -->
-  <xacro:macro name="zed_camera_description" params="prefix camera_name=zedm camera_model=zedm resolution=VGA">
-    <!--Camera-->
-    <!-- <joint name="${prefix}${camera_name}_camera_center_joint" type="fixed"> -->
-    <!--     <parent link="${prefix}${camera_name}_camera_mount_link"/> -->
-    <!--     <child link="${prefix}${camera_name}_camera_center"/> -->
-    <!--     <origin xyz="0.305 0 0.08" rpy="0 0 0" /> -->
-    <!-- </joint> -->
-    <!-- <link name="${prefix}${camera_name}_camera_center"> -->
-    <!--     <visual> -->
-    <!--         <origin xyz="0 0 0" rpy="0 0 0"/> -->
-    <!--         <geometry> -->
-    <!--             <mesh filename="file://$(find arcs_cohort_description)/meshes/zedm.stl"/> -->
-    <!--         </geometry> -->
-    <!--         <material name="black"> -->
-    <!--             <color rgba="0 0 0 0.9"/> -->
-    <!--         </material> -->
-    <!--     </visual> -->
-    <!-- </link> -->
-    <xacro:if value="${resolution == 'HD2K'}">
-        <xacro:property name="resolution_width" value="2208" />
-        <xacro:property name="resolution_height" value="1242" />
-        <xacro:property name="update_rate" value="15" />
-    </xacro:if>
-    <xacro:if value="${resolution == 'HD1080'}">
-        <xacro:property name="resolution_width" value="1920" />
-        <xacro:property name="resolution_height" value="1080" />
-        <xacro:property name="update_rate" value="30" />
-    </xacro:if>
-    <xacro:if value="${resolution == 'HD720'}">
-        <xacro:property name="resolution_width" value="1280" />
-        <xacro:property name="resolution_height" value="720" />
-        <xacro:property name="update_rate" value="60" />
-    </xacro:if>
-    <xacro:if value="${resolution == 'VGA'}">
-        <xacro:property name="resolution_width" value="672" />
-        <xacro:property name="resolution_height" value="376" />
-        <xacro:property name="update_rate" value="100" />
-    </xacro:if>
-    <xacro:if value="${camera_model == 'zed'}">
-        <xacro:property name="baseline" value="0.12" />
-        <xacro:property name="fov" value="2.0" />
-        <xacro:property name="clip_near" value="0.3" />
-        <xacro:property name="clip_far" value="25" />
-        <!-- Gazebo color -->
-        <gazebo reference="${camera_model}_camera_center">
-          <material>Gazebo/Grey</material>
+    <!-- Define a macro with a prefix param for the Zed M camera description -->
+    <xacro:macro name="zed_camera_description" params="prefix camera_name=zedm camera_model=zedm resolution=VGA">
+        <!-- Arguments for zed_wrapper/zed_camera -->
+        <xacro:arg name="custom_baseline"  default="0.0" />
+        <xacro:arg name="enable_gnss"   default="false" />
+        <xacro:arg name="gnss_x" default="0.0" />
+        <xacro:arg name="gnss_y" default="0.0" />
+        <xacro:arg name="gnss_z" default="0.0" />
+        <!-- Include zed_wrapper/zed_camera description -->
+        <xacro:include filename="$(find zed_wrapper)/urdf/zed_macro.urdf.xacro" />
+        <xacro:zed_camera name="$(arg camera_name)" model="$(arg camera_model)" custom_baseline="$(arg custom_baseline)" enable_gnss="$(arg enable_gnss)">
+                <origin xyz="$(arg gnss_x) $(arg gnss_y) $(arg gnss_z)" rpy="0 0 0"/>
+        </xacro:zed_camera>
+        <!--Camera-->
+        <joint name="${prefix}${camera_name}_camera_mount_to_camera" type="fixed">
+            <parent link="${prefix}${camera_name}_camera_mount_link"/>
+            <child link="${camera_name}_camera_link"/>
+            <origin xyz="0.037592 -0.0065 -0.02273" rpy="0 ${30*(M_PI/180)} 0" />
+        </joint>
+        <xacro:if value="${resolution == 'HD2K'}">
+            <xacro:property name="resolution_width" value="2208" />
+            <xacro:property name="resolution_height" value="1242" />
+            <xacro:property name="update_rate" value="15" />
+        </xacro:if>
+        <xacro:if value="${resolution == 'HD1080'}">
+            <xacro:property name="resolution_width" value="1920" />
+            <xacro:property name="resolution_height" value="1080" />
+            <xacro:property name="update_rate" value="30" />
+        </xacro:if>
+        <xacro:if value="${resolution == 'HD720'}">
+            <xacro:property name="resolution_width" value="1280" />
+            <xacro:property name="resolution_height" value="720" />
+            <xacro:property name="update_rate" value="60" />
+        </xacro:if>
+        <xacro:if value="${resolution == 'VGA'}">
+            <xacro:property name="resolution_width" value="672" />
+            <xacro:property name="resolution_height" value="376" />
+            <xacro:property name="update_rate" value="100" />
+        </xacro:if>
+        <xacro:if value="${camera_model == 'zed'}">
+            <xacro:property name="baseline" value="0.12" />
+            <xacro:property name="fov" value="2.0" />
+            <xacro:property name="clip_near" value="0.3" />
+            <xacro:property name="clip_far" value="25" />
+            <!-- Gazebo color -->
+            <gazebo reference="${camera_model}_camera_center">
+                <material>Gazebo/Grey</material>
+            </gazebo>
+        </xacro:if>
+        <xacro:if value="${camera_model == 'zedm'}">
+            <xacro:property name="baseline" value="0.06" />
+            <xacro:property name="fov" value="2.0" />
+            <xacro:property name="clip_near" value="0.1" />
+            <xacro:property name="clip_far" value="15" />
+            <!-- Add IMU for ZED -->
+            <!-- <xacro:imu_gazebo name="${camera_name}" frame="${camera_name}_imu_frame_gazebo" /> -->
+            <!-- Gazebo color -->
+            <gazebo reference="${camera_model}_camera_center">
+                <material>Gazebo/DarkGrey</material>
+            </gazebo>
+        </xacro:if>
+        <xacro:if value="${camera_model == 'zed2'}">
+            <xacro:property name="baseline" value="0.12" />
+            <xacro:property name="fov" value="1.8" />
+            <xacro:property name="clip_near" value="0.2" />
+            <xacro:property name="clip_far" value="20" />
+            <!-- Add IMU for ZED -->
+            <xacro:imu_gazebo name="${camera_name}" frame="${camera_name}_imu_frame_gazebo" />
+            <!-- Gazebo color -->
+            <gazebo reference="${camera_model}_camera_center">
+                <material>Gazebo/Black</material>
+            </gazebo>
+        </xacro:if>
+        <!-- Left Camera Gazebo -->
+        <gazebo reference="${camera_name}_left_camera_frame">
+            <sensor name="${prefix}left_camera" type="rgbd_camera">
+                <topic>camera/left_camera</topic>
+                <gz_frame_id>${camera_name}_left_camera_frame</gz_frame_id>
+                <always_on>1</always_on>
+                <update_rate>${update_rate}</update_rate>
+                <visualize>true</visualize>
+                <camera>
+                    <camera_info_topic>camera/left_camera_info</camera_info_topic>
+                    <horizontal_fov>${fov}</horizontal_fov>
+                    <image>
+                        <format>R8G8B8</format>
+                        <width>${resolution_width}</width>
+                        <height>${resolution_height}</height>
+                    </image>
+                    <clip>
+                        <near>${clip_near}</near>
+                        <far>${clip_far}</far>
+                    </clip>
+                </camera>
+            </sensor>
         </gazebo>
-    </xacro:if>
-    <xacro:if value="${camera_model == 'zedm'}">
-        <xacro:property name="baseline" value="0.06" />
-        <xacro:property name="fov" value="2.0" />
-        <xacro:property name="clip_near" value="0.1" />
-        <xacro:property name="clip_far" value="15" />
-        <!-- Add IMU for ZED -->
-        <!-- <xacro:imu_gazebo name="${camera_name}" frame="${camera_name}_imu_frame_gazebo" /> -->
-        <!-- Gazebo color -->
-        <gazebo reference="${camera_model}_camera_center">
-          <material>Gazebo/DarkGrey</material>
+        <!-- Right Camera Gazebo -->
+        <gazebo reference="${camera_name}_right_camera_frame">
+            <sensor name="${prefix}right_camera" type="camera">
+                <topic>camera/right_camera/image</topic>
+                <gz_frame_id>${camera_name}_right_camera_frame</gz_frame_id>
+                <visualize>true</visualize>
+                <update_rate>${update_rate}</update_rate>
+                <camera>
+                    <camera_info_topic>camera/right_camera/camera_info</camera_info_topic>
+                    <horizontal_fov>${fov}</horizontal_fov>
+                    <image>
+                        <format>R8G8B8</format>
+                        <width>${resolution_width}</width>
+                        <height>${resolution_height}</height>
+                    </image>
+                    <clip>
+                        <near>${clip_near}</near>
+                        <far>${clip_far}</far>
+                    </clip>
+                </camera>
+            </sensor>
         </gazebo>
-    </xacro:if>
-    <xacro:if value="${camera_model == 'zed2'}">
-        <xacro:property name="baseline" value="0.12" />
-        <xacro:property name="fov" value="1.8" />
-        <xacro:property name="clip_near" value="0.2" />
-        <xacro:property name="clip_far" value="20" />
-        <!-- Add IMU for ZED -->
-        <xacro:imu_gazebo name="${camera_name}" frame="${camera_name}_imu_frame_gazebo" />
-        <!-- Gazebo color -->
-        <gazebo reference="${camera_model}_camera_center">
-          <material>Gazebo/Black</material>
-        </gazebo>
-    </xacro:if>
-    <!-- Left Camera -->
-    <joint name="${prefix}${camera_name}_left_camera_joint" type="fixed">
-        <parent link="${prefix}${camera_name}_center_link"/>
-        <child link="${prefix}${camera_name}_left_camera_frame"/>
-        <origin xyz="0 ${baseline/2} 0" rpy="0 0 0" />
-    </joint>
-    <link name="${prefix}${camera_name}_left_camera_frame" />
-    <joint name="${prefix}${camera_name}_left_camera_optical_joint" type="fixed">
-        <parent link="${prefix}${camera_name}_left_camera_frame"/>
-        <child link="${prefix}${camera_name}_left_camera_optical_frame"/>
-        <!-- <origin xyz="0 0 0" rpy="-1.57079632679 0.0 -1.57079632679"/> -->
-        <origin xyz="0 0 0" rpy="0 0 0"/>
-    </joint>
-    <link name="${prefix}${camera_name}_left_camera_optical_frame"/>
-    <!-- Right Camera -->
-    <joint name="${prefix}${camera_name}_right_camera_joint" type="fixed">
-        <parent link="${prefix}${camera_name}_center_link"/>
-        <child link="${prefix}${camera_name}_right_camera_frame"/>
-        <origin xyz="0 -${baseline/2} 0" rpy="0 0 0" />
-    </joint>
-    <link name="${prefix}${camera_name}_right_camera_frame" />
-    <joint name="${prefix}${camera_name}_right_camera_optical_joint" type="fixed">
-        <parent link="${prefix}${camera_name}_right_camera_frame"/>
-        <child link="${prefix}${camera_name}_right_camera_optical_frame"/>
-        <!-- <origin xyz="0 0 0" rpy="-1.57079632679 0.0 -1.57079632679"/> -->
-        <origin xyz="0 0 0" rpy="0 0 0"/>
-    </joint>
-    <link name="${prefix}${camera_name}_right_camera_optical_frame"/>
-    <!-- Left Camera Gazebo -->
-    <gazebo reference="${prefix}${camera_name}_left_camera_frame">
-        <sensor name="${prefix}left_camera" type="rgbd_camera">
-            <topic>camera/left_camera</topic>
-            <gz_frame_id>${camera_name}_left_camera_optical_frame</gz_frame_id>
-            <always_on>1</always_on>
-            <update_rate>${update_rate}</update_rate>
-            <visualize>true</visualize>
-            <camera>
-                <camera_info_topic>camera/left_camera_info</camera_info_topic>
-                <horizontal_fov>${fov}</horizontal_fov>
-                <image>
-                    <format>R8G8B8</format>
-                    <width>${resolution_width}</width>
-                    <height>${resolution_height}</height>
-                </image>
-                <clip>
-                    <near>${clip_near}</near>
-                    <far>${clip_far}</far>
-                </clip>
-            </camera>
-        </sensor>
-    </gazebo>
-    <!-- Right Camera Gazebo -->
-    <gazebo reference="${prefix}${camera_name}_right_camera_frame">
-        <sensor name="${prefix}right_camera" type="camera">
-            <topic>camera/right_camera/image</topic>
-            <gz_frame_id>${camera_name}_right_camera_optical_frame</gz_frame_id>
-            <visualize>true</visualize>
-            <update_rate>${update_rate}</update_rate>
-            <camera>
-                <camera_info_topic>camera/right_camera/camera_info</camera_info_topic>
-                <horizontal_fov>${fov}</horizontal_fov>
-                <image>
-                    <format>R8G8B8</format>
-                    <width>${resolution_width}</width>
-                    <height>${resolution_height}</height>
-                </image>
-                <clip>
-                    <near>${clip_near}</near>
-                    <far>${clip_far}</far>
-                </clip>
-            </camera>
-        </sensor>
-    </gazebo>
-  </xacro:macro>
+    </xacro:macro>
 </robot>

Commit message: Add base_footprint

File: description/robot_core.xacro (robot description, xacro)
@@ -51,4 +51,11 @@
       </collision>
     </link>
+    <!-- Robot Footprint -->
+    <link name="${prefix}base_footprint"/>
+    <joint name="${prefix}base_joint" type="fixed">
+      <parent link="${prefix}base_link"/>
+      <child link="${prefix}base_footprint"/>
+      <origin xyz="0.0 0.0 -0.08" rpy="0 0 0"/>
+    </joint>
     <link name="${prefix}front_left_wheel_link">
       <inertial>

Commit message: Fix base_footprint z offset

File: description/robot_core.xacro (robot description, xacro)
@@ -3,4 +3,8 @@
   <!-- Define a macro with a prefix param for the robot description -->
   <xacro:macro name="robot_description" params="prefix camera_name=zedm camera_model=zedm">
+    <!-- Arguments -->
+    <xacro:property name="wheel_radius" value="0.08" />
+    <xacro:property name="base_footprint_z_offset" value="0.0295" />
+    <!-- Materials/Colors -->
     <material name="yellow">
       <color rgba="1 1 0 1"/>
@@ -56,5 +60,5 @@
       <parent link="${prefix}base_link"/>
       <child link="${prefix}base_footprint"/>
-      <origin xyz="0.0 0.0 -0.08" rpy="0 0 0"/>
+      <origin xyz="0.0 0.0 -${wheel_radius + base_footprint_z_offset}" rpy="0 0 0"/>
     </joint>
     <link name="${prefix}front_left_wheel_link">
