Commit message: fixed camera tf

File: description/robot.urdf.xacro (robot description, xacro)
@@ -2,3 +2,4 @@
 <robot xmlns:xacro="http://www.ros.org/wiki/xacro"  name="robot">
     <xacro:include filename="robot_core.xacro"/>
+    <xacro:include filename="zed_camera.xacro" />
 </robot>

File: description/zed_camera.xacro (robot description, xacro)
@@ -2,6 +2,6 @@
 <robot xmlns:xacro="http://www.ros.org/wiki/xacro" >
 <!--Camera-->
-    <joint name="zedm_camera_center_joint" type="fixed">
-        <parent link="chassis"/>
+    <!-- <joint name="zedm_camera_center_joint" type="fixed">
+        <parent link="zedmini_center_link"/>
         <child link="zedm_camera_center"/>
         <origin xyz="0.305 0 0.08" rpy="0 0 0" />
@@ -11,5 +11,4 @@
             <origin xyz="0 0 0" rpy="0 0 0"/>
             <geometry>
-            <!-- add zed camera stl -->
                 <mesh filename="file://$(find arcs_cohort_description)/meshes/zedm.stl"/>
             </geometry>
@@ -18,8 +17,8 @@
             </material>
         </visual>
-    </link>
+    </link> -->
     <!-- Left Camera -->
     <joint name="zedm_left_camera_joint" type="fixed">
-        <parent link="zedm_camera_center"/>
+        <parent link="zedmini_center_link"/>
         <child link="zedm_left_camera_frame"/>
         <origin xyz="0 0.03 0" rpy="0 0 0" />
@@ -34,5 +33,5 @@
     <!-- Right Camera -->
     <joint name="zedm_right_camera_joint" type="fixed">
-        <parent link="zedm_camera_center"/>
+        <parent link="zedmini_center_link"/>
         <child link="zedm_right_camera_frame"/>
         <origin xyz="0 -0.03 0" rpy="0 0 0" />
@@ -52,5 +51,5 @@
             <pose> 0 0 0 0 0 0 </pose>
             <visualize>true</visualize>
-            <update_rate>10</update_rate>
+            <update_rate>30</update_rate>
             <camera>
                 <camera_info_topic>camera/left_camera_info</camera_info_topic>
@@ -67,8 +66,5 @@
             </camera>
             <topic>camera/left_camera_image_raw</topic>
-            <gz_frame_id>camera_left_link_optical</gz_frame_id>
-            <!-- <plugin name="left_camera_controller" filename="libgazebo_ros_camera.so">
-                <frame_name>zedm_left_optical_frame</frame_name>
-            </plugin> -->
+            <gz_frame_id>zedm_left_camera_optical_frame</gz_frame_id>
         </sensor>
     </gazebo>
@@ -77,5 +73,5 @@
             <pose> 0 0 0 0 0 0 </pose>
             <visualize>true</visualize>
-            <update_rate>10</update_rate>
+            <update_rate>30</update_rate>
             <camera>
                 <camera_info_topic>camera/right_camera_info</camera_info_topic>
@@ -92,55 +88,6 @@
             </camera>
             <topic>camera/right_camera_image_raw</topic>
-            <gz_frame_id>camera_right_link_optical</gz_frame_id>
-            <!-- <plugin name="right_camera_controller" filename="libgazebo_ros_camera.so">
-                <frame_name>zedm_right_optical_frame</frame_name>
-            </plugin> -->
+            <gz_frame_id>zedm_right_camera_optical_frame</gz_frame_id>
         </sensor>
     </gazebo>
-    <!-- <gazebo reference="zedm_left_camera_frame">
-        <sensor type="multicamera" name="stereo_camera">
-        <visualize>true</visualize>
-          <update_rate>30.0</update_rate>
-          <camera name="left">
-            <horizontal_fov>1.089</horizontal_fov>
-            <image>
-              <width>640</width>
-              <height>800</height>
-              <format>R8G8B8</format>
-            </image>
-            <clip>
-              <near>0.05</near>
-              <far>8.0</far>
-            </clip>
-          </camera>
-          <camera name="right">
-            <pose>0 -0.06 0 0 0 0</pose>
-            <horizontal_fov>1.089</horizontal_fov>
-            <image>
-              <width>640</width>
-              <height>800</height>
-              <format>R8G8B8</format>
-            </image>
-            <clip>
-              <near>0.05</near>
-              <far>8.0</far>
-            </clip>
-          </camera>
-          <plugin name="stereo_camera_controller" filename="libgazebo_ros_multicamera.so">
-            <alwaysOn>true</alwaysOn>
-            <updateRate>30.0</updateRate>
-            <cameraName>multisense_sl/camera</cameraName>
-            <imageTopicName>image_raw</imageTopicName>
-            <cameraInfoTopicName>camera_info</cameraInfoTopicName>
-            <frameName>zedm_left_camera_optical_frame</frameName>
-            <rightFrameName>zedm_right_camera_optical_frame</rightFrameName>
-            <hackBaseline>0.06</hackBaseline>
-            <distortionK1>0.0</distortionK1>
-            <distortionK2>0.0</distortionK2>
-            <distortionK3>0.0</distortionK3>
-            <distortionT1>0.0</distortionT1>
-            <distortionT2>0.0</distortionT2>
-          </plugin>
-        </sensor>
-    </gazebo> -->
 </robot>

Commit message: added imu sim and gazebo diff drive xacro

File: description/robot.urdf.xacro (robot description, xacro)
@@ -2,4 +2,6 @@
 <robot xmlns:xacro="http://www.ros.org/wiki/xacro"  name="robot">
     <xacro:include filename="robot_core.xacro"/>
-    <xacro:include filename="zed_camera.xacro" />
+    <xacro:include filename="vectornav_imu.xacro"/>
+    <xacro:include filename="zed_camera.xacro"/>
+    <xacro:include filename="$(find arcs_cohort_gazebo_sim)/control/gazebo_diff_drive_plugin.xacro"/>
 </robot>

File: description/robot_core.xacro (robot description, xacro)
@@ -46,4 +46,5 @@
       <mesh
         filename="file://$(find arcs_cohort_description)/meshes/new_base_link.stl" />
+        <!-- <box size="0.28 0.13 0.08"/> -->
     </geometry>
   </collision>
@@ -82,4 +83,5 @@
       <mesh
         filename="file://$(find arcs_cohort_description)/meshes/new_front_left_wheel.stl" />
+      <!-- <sphere radius="0.08"/> -->
     </geometry>
   </collision>
@@ -131,4 +133,5 @@
       <mesh
         filename="file://$(find arcs_cohort_description)/meshes/new_front_right_wheel.stl" />
+      <!-- <sphere radius="0.08"/> -->
     </geometry>
   </collision>
@@ -180,4 +183,5 @@
       <mesh
         filename="file://$(find arcs_cohort_description)/meshes/new_back_left_wheel.stl" />
+      <!-- <sphere radius="0.08"/> -->
     </geometry>
   </collision>
@@ -229,4 +233,5 @@
       <mesh
         filename="file://$(find arcs_cohort_description)/meshes/new_back_right_wheel.stl" />
+      <!-- <sphere radius="0.08"/> -->
     </geometry>
   </collision>
@@ -282,4 +287,5 @@
       <mesh
         filename="file://$(find arcs_cohort_description)/meshes/new_imu.stl" />
+      <!-- <box size = "0.03 0.025 0.01"/> -->
     </geometry>
   </collision>
@@ -331,4 +337,5 @@
       <mesh
         filename="file://$(find arcs_cohort_description)/meshes/new_camera_mount.stl" />
+      <!-- <box size="0.05 0.115 0.05" /> -->
     </geometry>
   </collision>
@@ -381,4 +388,5 @@
       <mesh
         filename="file://$(find arcs_cohort_description)/meshes/zedmini_center_link.STL" />
+      <!-- <box size="0.015 0.122 0.025"/> -->
     </geometry>
   </collision>

File: description/zed_camera.xacro (robot description, xacro)
@@ -44,7 +44,7 @@
     </joint>
     <link name="zedm_right_camera_optical_frame"/>
-    <gazebo reference="zedm_camera_center">
+    <!-- <gazebo reference="zedm_camera_center">
         <material>Gazebo/Green</material>
-    </gazebo>
+    </gazebo> -->
     <gazebo reference="zedm_left_camera_frame">
         <sensor name="left_camera" type="camera">

Commit message: Add prefix arg to xacros

File: description/robot.urdf.xacro (robot description, xacro)
@@ -1,7 +1,16 @@
 <?xml version="1.0"?>
-<robot xmlns:xacro="http://www.ros.org/wiki/xacro"  name="robot">
+<robot xmlns:xacro="http://www.ros.org/wiki/xacro" name="robot">
+    <!-- Define the prefix property -->
+    <xacro:arg name="prefix" default="" />
+    <!-- Include robot components -->
     <xacro:include filename="robot_core.xacro"/>
     <xacro:include filename="vectornav_imu.xacro"/>
     <xacro:include filename="zed_camera.xacro"/>
+    <!-- Include Gazebo plugins -->
     <xacro:include filename="$(find arcs_cohort_gazebo_sim)/control/gazebo_diff_drive_plugin.xacro"/>
+    <!-- Call the robot description macro with the prefix -->
+    <xacro:robot_description prefix="$(arg prefix)"/>
+    <xacro:vectornav_imu_description prefix="$(arg prefix)"/>
+    <xacro:zed_camera_description prefix="$(arg prefix)"/>
+    <xacro:gazebo_diff_drive_plugin_description prefix="$(arg prefix)"/>
 </robot>

File: description/robot_core.xacro (robot description, xacro)
@@ -1,407 +1,350 @@
 <?xml version="1.0"?>
 <robot xmlns:xacro="http://www.ros.org/wiki/xacro">
-  <material name="yellow">
+  <!-- Define a macro with a prefix param for the robot description -->
+  <xacro:macro name="robot_description" params="prefix">
+    <material name="yellow">
       <color rgba="1 1 0 1"/>
-  </material>
-  <material name="orange">
+    </material>
+    <material name="orange">
       <color rgba="1 0.3 0.1 1"/>
-  </material>
-  <material name="blue">
+    </material>
+    <material name="blue">
       <color rgba="0.2 0.2 1 1"/>
-  </material>
-  <material name="red">
+    </material>
+    <material name="red">
       <color rgba="1 0 0 1"/>
-  </material>
-  <link
-  name="base_link">
-  <inertial>
-    <origin
-      xyz="0.00180125809402712 0.000803676445247231 0.01518679730351"
-      rpy="0 0 0" />
-    <mass
-      value="0.657677203206575" />
-    <inertia
-      ixx="0.00086538199329254"
-      ixy="-2.9353575955111E-07"
-      ixz="2.01709713615107E-05"
-      iyy="0.00372020827025877"
-      iyz="-4.62454840349382E-06"
-      izz="0.00438426362438441" />
-  </inertial>
-  <visual>
-    <origin
-      xyz="0 0 0"
-      rpy="0 0 0" />
-    <geometry>
-        <mesh
-        filename="file://$(find arcs_cohort_description)/meshes/new_base_link.stl"/>
-    </geometry>
-    <material name="blue"/>
-  </visual>
-  <collision>
-    <origin
-      xyz="0 0 0"
-      rpy="0 0 0" />
-    <geometry>
-      <mesh
-        filename="file://$(find arcs_cohort_description)/meshes/new_base_link.stl" />
-        <!-- <box size="0.28 0.13 0.08"/> -->
-    </geometry>
-  </collision>
-</link>
-<link
-  name="front_left_wheel_link">
-  <inertial>
-    <origin
-      xyz="-2.6737853597858E-10 1.57494023378391E-09 0.00586031499671241"
-      rpy="0 0 0" />
-    <mass
-      value="0.0636859538546401" />
-    <inertia
-      ixx="0.000148107353320268"
-      ixy="-1.35785185033322E-11"
-      ixz="4.45745626426646E-12"
-      iyy="0.000148107350264006"
-      iyz="1.98277930663145E-12"
-      izz="0.000285045799220755" />
-  </inertial>
-  <visual>
-    <origin
-      xyz="0 0 0"
-      rpy="0 0 0" />
-    <geometry>
-      <mesh
-        filename="file://$(find arcs_cohort_description)/meshes/new_front_left_wheel.stl" />
-    </geometry>
-    <material name="orange"/>
-  </visual>
-  <collision>
-    <origin
-      xyz="0 0 0"
-      rpy="0 0 0" />
-    <geometry>
-      <mesh
-        filename="file://$(find arcs_cohort_description)/meshes/new_front_left_wheel.stl" />
-      <!-- <sphere radius="0.08"/> -->
-    </geometry>
-  </collision>
-</link>
-<joint
-  name="front_left_wheel_joint"
-  type="continuous">
-  <origin
-    xyz="0.12851 0.11738 -0.022625"
-    rpy="-1.5708 0 0" />
-  <parent
-    link="base_link" />
-  <child
-    link="front_left_wheel_link" />
-  <axis
-    xyz="0 0 1" />
-</joint>
-<link
-  name="front_right_wheel_link">
-  <inertial>
-    <origin
-      xyz="-1.3376E-09 -8.8541E-10 0.0058603"
-      rpy="0 0 0" />
-    <mass
-      value="0.063686" />
-    <inertia
-      ixx="0.00014811"
-      ixy="-5.3705E-12"
-      ixz="-3.5018E-12"
-      iyy="0.00014811"
-      iyz="3.3368E-12"
-      izz="0.00028505" />
-  </inertial>
-  <visual>
-    <origin
-      xyz="0 0 0"
-      rpy="0 0 0" />
-    <geometry>
-      <mesh
-        filename="file://$(find arcs_cohort_description)/meshes/new_front_right_wheel.stl" />
-    </geometry>
-    <material name="orange"/>
-  </visual>
-  <collision>
-    <origin
-      xyz="0 0 0"
-      rpy="0 0 0" />
-    <geometry>
-      <mesh
-        filename="file://$(find arcs_cohort_description)/meshes/new_front_right_wheel.stl" />
-      <!-- <sphere radius="0.08"/> -->
-    </geometry>
-  </collision>
-</link>
-<joint
-  name="front_right_wheel_joint"
-  type="continuous">
-  <origin
-    xyz="0.12051 -0.11682 -0.022625"
-    rpy="1.5708 0 0" />
-  <parent
-    link="base_link" />
-  <child
-    link="front_right_wheel_link" />
-  <axis
-    xyz="0 0 -1" />
-</joint>
-<link
-  name="back_left_wheel_link">
-  <inertial>
-    <origin
-      xyz="-9.53E-10 -1.113E-09 0.0058603"
-      rpy="0 0 0" />
-    <mass
-      value="0.063686" />
-    <inertia
-      ixx="0.00014811"
-      ixy="-4.9708E-12"
-      ixz="-4.0149E-12"
-      iyy="0.00014811"
-      iyz="1.9832E-12"
-      izz="0.00028505" />
-  </inertial>
-  <visual>
-    <origin
-      xyz="0 0 0"
-      rpy="0 0 0" />
-    <geometry>
-      <mesh
-        filename="file://$(find arcs_cohort_description)/meshes/new_back_left_wheel.stl" />
-    </geometry>
-    <material name="orange"/>
-  </visual>
-  <collision>
-    <origin
-      xyz="0 0 0"
-      rpy="0 0 0" />
-    <geometry>
-      <mesh
-        filename="file://$(find arcs_cohort_description)/meshes/new_back_left_wheel.stl" />
-      <!-- <sphere radius="0.08"/> -->
-    </geometry>
-  </collision>
-</link>
-<joint
-  name="back_left_wheel_joint"
-  type="continuous">
-  <origin
-    xyz="-0.11949 0.11738 -0.022625"
-    rpy="-1.5708 0 0" />
-  <parent
-    link="base_link" />
-  <child
-    link="back_left_wheel_link" />
-  <axis
-    xyz="0 0 1" />
-</joint>
-<link
-  name="back_right_wheel_link">
-  <inertial>
-    <origin
-      xyz="-3.4938159310105E-10 -6.88384349523119E-11 0.00586031504576194"
-      rpy="0 0 0" />
-    <mass
-      value="0.063685952885413" />
-    <inertia
-      ixx="0.000148107341904413"
-      ixy="-9.56591142331185E-12"
-      ixz="-4.24605263320539E-13"
-      iyy="0.000148107361436709"
-      iyz="9.18578002146026E-13"
-      izz="0.000285045798997703" />
-  </inertial>
-  <visual>
-    <origin
-      xyz="0 0 0"
-      rpy="0 0 0" />
-    <geometry>
-      <mesh
-        filename="file://$(find arcs_cohort_description)/meshes/new_back_right_wheel.stl" />
-    </geometry>
-    <material name="orange"/>
-  </visual>
-  <collision>
-    <origin
-      xyz="0 0 0"
-      rpy="0 0 0" />
-    <geometry>
-      <mesh
-        filename="file://$(find arcs_cohort_description)/meshes/new_back_right_wheel.stl" />
-      <!-- <sphere radius="0.08"/> -->
-    </geometry>
-  </collision>
-</link>
-<joint
-  name="back_right_wheel_joint"
-  type="continuous">
-  <origin
-    xyz="-0.12749 -0.11682 -0.022625"
-    rpy="1.5708 0 0" />
-  <parent
-    link="base_link" />
-  <child
-    link="back_right_wheel_link" />
-  <axis
-    xyz="0 0 -1" />
-</joint>
-<link
-  name="imu_link">
-  <inertial>
-    <origin
-      xyz="-0.000894812057582933 9.60259274576658E-06 -0.00456943294796108"
-      rpy="0 0 0" />
-    <mass
-      value="0.0065760792742103" />
-    <inertia
-      ixx="3.78511408547619E-07"
-      ixy="4.67820105640642E-11"
-      ixz="1.00912927862616E-08"
-      iyy="3.79926110271894E-07"
-      iyz="-5.01543493566598E-12"
-      izz="7.19032056380139E-07" />
-  </inertial>
-  <visual>
-    <origin
-      xyz="0 0 0"
-      rpy="0 0 0" />
-    <geometry>
-      <mesh
-        filename="file://$(find arcs_cohort_description)/meshes/new_imu.stl" />
-    </geometry>
-    <material
-      name="">
-      <color
-        rgba="0.792156862745098 0.819607843137255 0.933333333333333 1" />
     </material>
-  </visual>
-  <collision>
-    <origin
-      xyz="0 0 0"
-      rpy="0 0 0" />
-    <geometry>
-      <mesh
-        filename="file://$(find arcs_cohort_description)/meshes/new_imu.stl" />
-      <!-- <box size = "0.03 0.025 0.01"/> -->
-    </geometry>
-  </collision>
-</link>
-<joint
-  name="imu_joint"
-  type="fixed">
-  <origin
-    xyz="0.0022791 0.00028171 0.01489"
-    rpy="0 0 0" />
-  <parent
-    link="base_link" />
-  <child
-    link="imu_link" />
-  <axis
-    xyz="0 0 0" />
-</joint>
-<link
-  name="camera_mount_link">
-  <inertial>
-    <origin
-      xyz="0 0 0"
-      rpy="0 0 0" />
-    <mass
-      value="0" />
-    <inertia
-      ixx="0"
-      ixy="0"
-      ixz="0"
-      iyy="0"
-      iyz="0"
-      izz="0" />
-  </inertial>
-  <visual>
-    <origin
-      xyz="0 0 0"
-      rpy="0 0 0" />
-    <geometry>
-      <mesh
-        filename="file://$(find arcs_cohort_description)/meshes/new_camera_mount.stl" />
-    </geometry>
-    <material name="red"/>
-  </visual>
-  <collision>
-    <origin
-      xyz="0 0 0"
-      rpy="0 0 0" />
-    <geometry>
-      <mesh
-        filename="file://$(find arcs_cohort_description)/meshes/new_camera_mount.stl" />
-      <!-- <box size="0.05 0.115 0.05" /> -->
-    </geometry>
-  </collision>
-</link>
-<joint
-  name="camera_mount_joint"
-  type="fixed">
-  <origin
-    xyz="0.14426 0.00028171 0.094535"
-    rpy="0 0 0" />
-  <parent
-    link="base_link" />
-  <child
-    link="camera_mount_link" />
-  <axis
-    xyz="0 0 0" />
-</joint>
-<link
-  name="zedmini_center_link">
-  <inertial>
-    <origin
-      xyz="-0.00435147007919079 -0.00309486253694627 0.00251127017920943"
-      rpy="0 0 0" />
-    <mass
-      value="0.0560548842495178" />
-    <inertia
-      ixx="7.29762807495571E-05"
-      ixy="5.57132554461124E-07"
-      ixz="-2.34695280152666E-07"
-      iyy="5.49793925654236E-06"
-      iyz="-3.21584411064254E-07"
-      izz="7.2705806093778E-05" />
-  </inertial>
-  <visual>
-    <origin
-      xyz="0 0 0"
-      rpy="0 0 0" />
-    <geometry>
-      <mesh
-        filename="file://$(find arcs_cohort_description)/meshes/zedmini_center_link.STL" />
-    </geometry>
-    <material
-      name="yellow"/>
-  </visual>
-  <collision>
-    <origin
-      xyz="0 0 0"
-      rpy="0 0 0" />
-    <geometry>
-      <mesh
-        filename="file://$(find arcs_cohort_description)/meshes/zedmini_center_link.STL" />
-      <!-- <box size="0.015 0.122 0.025"/> -->
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
File: description/vectornav_imu.xacro (robot description, xacro)
@@ -1,5 +1,7 @@
 <?xml version="1.0"?>
 <robot xmlns:xacro="http://www.ros.org/wiki/xacro" >
-    <gazebo reference="imu_link">
+  <!-- Define a macro with a prefix param for the VectorNav IMU description -->
+  <xacro:macro name="vectornav_imu_description" params="prefix">
+    <gazebo reference="${prefix}imu_link">
         <sensor name="vn100_imu" type="imu">
             <always_on>true</always_on>
@@ -50,3 +52,4 @@
         </sensor>
     </gazebo>
+  </xacro:macro>
 </robot>

File: description/zed_camera.xacro (robot description, xacro)
@@ -1,11 +1,13 @@
 <?xml version="1.0"?>
 <robot xmlns:xacro="http://www.ros.org/wiki/xacro" >
+  <!-- Define a macro with a prefix param for the Zed M camera description -->
+  <xacro:macro name="zed_camera_description" params="prefix">
     <!--Camera-->
-    <!-- <joint name="zedm_camera_center_joint" type="fixed">
-        <parent link="zedmini_center_link"/>
-        <child link="zedm_camera_center"/>
+    <!-- <joint name="${prefix}zedm_camera_center_joint" type="fixed">
+        <parent link="${prefix}zedmini_center_link"/>
+        <child link="${prefix}zedm_camera_center"/>
         <origin xyz="0.305 0 0.08" rpy="0 0 0" />
     </joint>
-    <link name="zedm_camera_center">
+    <link name="${prefix}zedm_camera_center">
         <visual>
             <origin xyz="0 0 0" rpy="0 0 0"/>
@@ -19,34 +21,34 @@
     </link> -->
     <!-- Left Camera -->
-    <joint name="zedm_left_camera_joint" type="fixed">
-        <parent link="zedmini_center_link"/>
-        <child link="zedm_left_camera_frame"/>
+    <joint name="${prefix}zedm_left_camera_joint" type="fixed">
+        <parent link="${prefix}zedmini_center_link"/>
+        <child link="${prefix}zedm_left_camera_frame"/>
         <origin xyz="0 0.03 0" rpy="0 0 0" />
     </joint>
-    <link name="zedm_left_camera_frame" />
-    <joint name="zedm_left_camera_optical_joint" type="fixed">
+    <link name="${prefix}zedm_left_camera_frame" />
+    <joint name="${prefix}zedm_left_camera_optical_joint" type="fixed">
         <origin xyz="0 0 0" rpy="-1.57079632679 0.0 -1.57079632679"/>
-        <parent link="zedm_left_camera_frame"/>
-        <child link="zedm_left_camera_optical_frame"/>
+        <parent link="${prefix}zedm_left_camera_frame"/>
+        <child link="${prefix}zedm_left_camera_optical_frame"/>
     </joint>
-    <link name="zedm_left_camera_optical_frame"/>
+    <link name="${prefix}zedm_left_camera_optical_frame"/>
     <!-- Right Camera -->
-    <joint name="zedm_right_camera_joint" type="fixed">
-        <parent link="zedmini_center_link"/>
-        <child link="zedm_right_camera_frame"/>
+    <joint name="${prefix}zedm_right_camera_joint" type="fixed">
+        <parent link="${prefix}zedmini_center_link"/>
+        <child link="${prefix}zedm_right_camera_frame"/>
         <origin xyz="0 -0.03 0" rpy="0 0 0" />
     </joint>
-    <link name="zedm_right_camera_frame" />
-    <joint name="zedm_right_camera_optical_joint" type="fixed">
+    <link name="${prefix}zedm_right_camera_frame" />
+    <joint name="${prefix}zedm_right_camera_optical_joint" type="fixed">
         <origin xyz="0 0 0" rpy="-1.57079632679 0.0 -1.57079632679"/>
-        <parent link="zedm_right_camera_frame"/>
-        <child link="zedm_right_camera_optical_frame"/>
+        <parent link="${prefix}zedm_right_camera_frame"/>
+        <child link="${prefix}zedm_right_camera_optical_frame"/>
     </joint>
-    <link name="zedm_right_camera_optical_frame"/>
-    <!-- <gazebo reference="zedm_camera_center">
+    <link name="${prefix}zedm_right_camera_optical_frame"/>
+    <!-- <gazebo reference="${prefix}zedm_camera_center">
         <material>Gazebo/Green</material>
     </gazebo> -->
-    <gazebo reference="zedm_left_camera_frame">
-        <sensor name="left_camera" type="camera">
+    <gazebo reference="${prefix}zedm_left_camera_frame">
+        <sensor name="${prefix}left_camera" type="camera">
             <pose> 0 0 0 0 0 0 </pose>
             <visualize>true</visualize>
@@ -69,6 +71,6 @@
         </sensor>
     </gazebo>
-    <gazebo reference="zedm_right_camera_frame">
-        <sensor name="right_camera" type="camera">
+    <gazebo reference="${prefix}zedm_right_camera_frame">
+        <sensor name="${prefix}right_camera" type="camera">
             <pose> 0 0 0 0 0 0 </pose>
             <visualize>true</visualize>
@@ -91,3 +93,4 @@
         </sensor>
     </gazebo>
+  </xacro:macro>
 </robot>
