Commit message: Add camera resolution params

File: description/robot.urdf.xacro (robot description, xacro)
@@ -3,4 +3,5 @@
     <!-- Define the prefix property -->
     <xacro:arg name="prefix" default="" />
+    <xacro:arg name="camera_resolution" default="HD720" />
     <!-- Include robot components -->
     <xacro:include filename="robot_core.xacro"/>
@@ -12,5 +13,5 @@
     <xacro:robot_description prefix="$(arg prefix)"/>
     <xacro:vectornav_imu_description prefix="$(arg prefix)"/>
-    <xacro:zed_camera_description prefix="$(arg prefix)"/>
+    <xacro:zed_camera_description prefix="$(arg prefix)" resolution="$(arg camera_resolution)"/>
     <xacro:gazebo_diff_drive_plugin_description prefix="$(arg prefix)"/>
 </robot>

File: description/zed_camera.xacro (robot description, xacro)
@@ -1,6 +1,12 @@
 <?xml version="1.0"?>
+<!--
+Stereolabs Zed Camera Model
+Borrows from:
+https://github.com/stereolabs/zed-ros2-wrapper/tree/master/zed_wrapper/urdf
+https://github.com/rpanther/panther_simulation/blob/master/panther_gazebo/urdf
+-->
 <robot xmlns:xacro="http://www.ros.org/wiki/xacro" >
   <!-- Define a macro with a prefix param for the Zed M camera description -->
-  <xacro:macro name="zed_camera_description" params="prefix">
+  <xacro:macro name="zed_camera_description" params="prefix resolution=VGA">
     <!--Camera-->
     <!-- <joint name="${prefix}zedm_camera_center_joint" type="fixed">
@@ -20,4 +26,24 @@
         </visual>
     </link> -->
+    <xacro:if value="${resolution == 'HD2K'}">
+        <xacro:property name="resolution_width" value="2208" />
+        <xacro:property name="resolution_height" value="1242" />
+        <xacro:property name="update_rate" value="15" />
+    </xacro:if>
+    <xacro:if value="${resolution == 'HD1080'}">
+        <xacro:property name="resolution_width" value="1920" />
+        <xacro:property name="resolution_height" value="1080" />
+        <xacro:property name="update_rate" value="30" />
+    </xacro:if>
+    <xacro:if value="${resolution == 'HD720'}">
+        <xacro:property name="resolution_width" value="1280" />
+        <xacro:property name="resolution_height" value="720" />
+        <xacro:property name="update_rate" value="60" />
+    </xacro:if>
+    <xacro:if value="${resolution == 'VGA'}">
+        <xacro:property name="resolution_width" value="672" />
+        <xacro:property name="resolution_height" value="376" />
+        <xacro:property name="update_rate" value="100" />
+    </xacro:if>
     <!-- Left Camera -->
     <joint name="${prefix}zedm_left_camera_joint" type="fixed">
@@ -53,5 +79,5 @@
             <pose> 0 0 0 0 0 0 </pose>
             <visualize>true</visualize>
-            <update_rate>30</update_rate>
+            <update_rate>${update_rate}</update_rate>
             <camera>
                 <camera_info_topic>camera/left_camera_info</camera_info_topic>
@@ -59,6 +85,6 @@
                 <image>
                     <format>R8G8B8</format>
-                    <width>640</width>
-                    <height>480</height>
+                    <width>${resolution_width}</width>
+                    <height>${resolution_height}</height>
                 </image>
                 <clip>
@@ -75,5 +101,5 @@
             <pose> 0 0 0 0 0 0 </pose>
             <visualize>true</visualize>
-            <update_rate>30</update_rate>
+            <update_rate>${update_rate}</update_rate>
             <camera>
                 <camera_info_topic>camera/right_camera_info</camera_info_topic>
@@ -81,6 +107,6 @@
                 <image>
                     <format>R8G8B8</format>
-                    <width>640</width>
-                    <height>480</height>
+                    <width>${resolution_width}</width>
+                    <height>${resolution_height}</height>
                 </image>
                 <clip>

Commit message: Add camera name/model parameterization

File: description/robot.urdf.xacro (robot description, xacro)
@@ -3,4 +3,6 @@
     <!-- Define the prefix property -->
     <xacro:arg name="prefix" default="" />
+    <xacro:arg name="camera_name" default="zedm" />
+    <xacro:arg name="camera_model" default="zedm" />
     <xacro:arg name="camera_resolution" default="HD720" />
     <!-- Include robot components -->
@@ -11,7 +13,7 @@
     <xacro:include filename="$(find arcs_cohort_gazebo_sim)/control/gazebo_diff_drive_plugin.xacro"/>
     <!-- Call the robot description macro with the prefix -->
-    <xacro:robot_description prefix="$(arg prefix)"/>
+    <xacro:robot_description prefix="$(arg prefix)" camera_name="$(arg camera_name)" camera_model="$(arg camera_model)"/>
     <xacro:vectornav_imu_description prefix="$(arg prefix)"/>
-    <xacro:zed_camera_description prefix="$(arg prefix)" resolution="$(arg camera_resolution)"/>
+    <xacro:zed_camera_description prefix="$(arg prefix)" camera_name="$(arg camera_name)" camera_model="$(arg camera_model)" resolution="$(arg camera_resolution)"/>
     <xacro:gazebo_diff_drive_plugin_description prefix="$(arg prefix)"/>
 </robot>

File: description/robot_core.xacro (robot description, xacro)
@@ -2,5 +2,5 @@
 <robot xmlns:xacro="http://www.ros.org/wiki/xacro">
   <!-- Define a macro with a prefix param for the robot description -->
-  <xacro:macro name="robot_description" params="prefix">
+  <xacro:macro name="robot_description" params="prefix camera_name=zedm camera_model=zedm">
     <material name="yellow">
       <color rgba="1 1 0 1"/>
@@ -307,5 +307,5 @@
       <axis xyz="0 0 0" />
     </joint>
-    <link name="${prefix}zedmini_center_link">
+    <link name="${prefix}${camera_name}_center_link">
       <inertial>
         <origin xyz="-0.00435147007919079 -0.00309486253694627 0.00251127017920943" rpy="0 0 0" />
@@ -325,5 +325,5 @@
         <geometry>
           <mesh
-            filename="file://$(find arcs_cohort_description)/meshes/zedmini_center_link.STL" />
+            filename="file://$(find arcs_cohort_description)/meshes/${camera_model}_center_link.STL" />
         </geometry>
         <material
@@ -336,13 +336,13 @@
         <geometry>
           <mesh
-            filename="file://$(find arcs_cohort_description)/meshes/zedmini_center_link.STL" />
+            filename="file://$(find arcs_cohort_description)/meshes/${camera_model}_center_link.STL" />
           <!-- <box size="0.015 0.122 0.025"/> -->
         </geometry>
       </collision>
     </link>
-    <joint name="${prefix}zedmini_center_joint" type="fixed">
+    <joint name="${prefix}${camera_name}_center_joint" type="fixed">
       <origin xyz="0.050151 0.0018215 -0.015053" rpy="0 0 0" />
       <parent link="${prefix}camera_mount_link" />
-      <child link="${prefix}zedmini_center_link" />
+      <child link="${prefix}${camera_name}_center_link" />
       <axis xyz="0 0 0" />
     </joint>

File: description/zed_camera.xacro (robot description, xacro)
@@ -8,5 +8,5 @@
 <robot xmlns:xacro="http://www.ros.org/wiki/xacro" >
   <!-- Define a macro with a prefix param for the Zed M camera description -->
-  <xacro:macro name="zed_camera_description" params="prefix resolution=VGA">
+  <xacro:macro name="zed_camera_description" params="prefix camera_name=zedm camera_model=zedm resolution=VGA">
     <!--Camera-->
     <!-- <joint name="${prefix}zedm_camera_center_joint" type="fixed">
@@ -46,36 +46,71 @@
         <xacro:property name="update_rate" value="100" />
     </xacro:if>
+    <xacro:if value="${camera_model == 'zed'}">
+        <xacro:property name="baseline" value="0.12" />
+        <xacro:property name="fov" value="2.0" />
+        <xacro:property name="clip_near" value="0.3" />
+        <xacro:property name="clip_far" value="25" />
+        <!-- Gazebo color -->
+        <gazebo reference="${camera_model}_camera_center">
+          <material>Gazebo/Grey</material>
+        </gazebo>
+    </xacro:if>
+    <xacro:if value="${camera_model == 'zedm'}">
+        <xacro:property name="baseline" value="0.06" />
+        <xacro:property name="fov" value="2.0" />
+        <xacro:property name="clip_near" value="0.1" />
+        <xacro:property name="clip_far" value="15" />
+        <!-- Add IMU for ZED -->
+        <!-- <xacro:imu_gazebo name="${camera_name}" frame="${camera_name}_imu_frame_gazebo" /> -->
+        <!-- Gazebo color -->
+        <gazebo reference="${camera_model}_camera_center">
+          <material>Gazebo/DarkGrey</material>
+        </gazebo>
+    </xacro:if>
+    <xacro:if value="${camera_model == 'zed2'}">
+        <xacro:property name="baseline" value="0.12" />
+        <xacro:property name="fov" value="1.8" />
+        <xacro:property name="clip_near" value="0.2" />
+        <xacro:property name="clip_far" value="20" />
+        <!-- Add IMU for ZED -->
+        <xacro:imu_gazebo name="${camera_name}" frame="${camera_name}_imu_frame_gazebo" />
+        <!-- Gazebo color -->
+        <gazebo reference="${camera_model}_camera_center">
+          <material>Gazebo/Black</material>
+        </gazebo>
+    </xacro:if>
     <!-- Left Camera -->
-    <joint name="${prefix}zedm_left_camera_joint" type="fixed">
-        <parent link="${prefix}zedmini_center_link"/>
-        <child link="${prefix}zedm_left_camera_frame"/>
-        <origin xyz="0 0.03 0" rpy="0 0 0" />
+    <joint name="${prefix}${camera_name}_left_camera_joint" type="fixed">
+        <parent link="${prefix}${camera_name}_center_link"/>
+        <child link="${prefix}${camera_name}_left_camera_frame"/>
+        <origin xyz="0 ${baseline/2} 0" rpy="0 0 0" />
     </joint>
-    <link name="${prefix}zedm_left_camera_frame" />
-    <joint name="${prefix}zedm_left_camera_optical_joint" type="fixed">
-        <parent link="${prefix}zedm_left_camera_frame"/>
-        <child link="${prefix}zedm_left_camera_optical_frame"/>
+    <link name="${prefix}${camera_name}_left_camera_frame" />
+    <joint name="${prefix}${camera_name}_left_camera_optical_joint" type="fixed">
+        <parent link="${prefix}${camera_name}_left_camera_frame"/>
+        <child link="${prefix}${camera_name}_left_camera_optical_frame"/>
         <!-- <origin xyz="0 0 0" rpy="-1.57079632679 0.0 -1.57079632679"/> -->
         <origin xyz="0 0 0" rpy="0 0 0"/>
     </joint>
-    <link name="${prefix}zedm_left_camera_optical_frame"/>
+    <link name="${prefix}${camera_name}_left_camera_optical_frame"/>
     <!-- Right Camera -->
-    <joint name="${prefix}zedm_right_camera_joint" type="fixed">
-        <parent link="${prefix}zedmini_center_link"/>
-        <child link="${prefix}zedm_right_camera_frame"/>
-        <origin xyz="0 -0.03 0" rpy="0 0 0" />
+    <joint name="${prefix}${camera_name}_right_camera_joint" type="fixed">
+        <parent link="${prefix}${camera_name}_center_link"/>
+        <child link="${prefix}${camera_name}_right_camera_frame"/>
+        <origin xyz="0 -${baseline/2} 0" rpy="0 0 0" />
     </joint>
-    <link name="${prefix}zedm_right_camera_frame" />
-    <joint name="${prefix}zedm_right_camera_optical_joint" type="fixed">
-        <parent link="${prefix}zedm_right_camera_frame"/>
-        <child link="${prefix}zedm_right_camera_optical_frame"/>
-        <origin xyz="0 0 0" rpy="-1.57079632679 0.0 -1.57079632679"/>
+    <link name="${prefix}${camera_name}_right_camera_frame" />
+    <joint name="${prefix}${camera_name}_right_camera_optical_joint" type="fixed">
+        <parent link="${prefix}${camera_name}_right_camera_frame"/>
+        <child link="${prefix}${camera_name}_right_camera_optical_frame"/>
+        <!-- <origin xyz="0 0 0" rpy="-1.57079632679 0.0 -1.57079632679"/> -->
+        <origin xyz="0 0 0" rpy="0 0 0"/>
     </joint>
-    <link name="${prefix}zedm_right_camera_optical_frame"/>
+    <link name="${prefix}${camera_name}_right_camera_optical_frame"/>
     <!-- Left Camera Gazebo -->
-    <gazebo reference="${prefix}zedm_left_camera_frame">
+    <gazebo reference="${prefix}${camera_name}_left_camera_frame">
         <sensor name="${prefix}left_camera" type="rgbd_camera">
             <topic>camera/left_camera</topic>
-            <gz_frame_id>zedm_left_camera_optical_frame</gz_frame_id>
+            <gz_frame_id>${camera_name}_left_camera_optical_frame</gz_frame_id>
             <always_on>1</always_on>
             <update_rate>${update_rate}</update_rate>
@@ -83,5 +118,5 @@
             <camera>
                 <camera_info_topic>camera/left_camera_info</camera_info_topic>
-                <horizontal_fov>1.089</horizontal_fov>
+                <horizontal_fov>${fov}</horizontal_fov>
                 <image>
                     <format>R8G8B8</format>
@@ -90,6 +125,6 @@
                 </image>
                 <clip>
-                    <near>0.05</near>
-                    <far>8.0</far>
+                    <near>${clip_near}</near>
+                    <far>${clip_far}</far>
                 </clip>
             </camera>
@@ -97,13 +132,13 @@
     </gazebo>
     <!-- Right Camera Gazebo -->
-    <gazebo reference="${prefix}zedm_right_camera_frame">
+    <gazebo reference="${prefix}${camera_name}_right_camera_frame">
         <sensor name="${prefix}right_camera" type="camera">
             <topic>camera/right_camera/image</topic>
-            <gz_frame_id>zedm_right_camera_optical_frame</gz_frame_id>
+            <gz_frame_id>${camera_name}_right_camera_optical_frame</gz_frame_id>
             <visualize>true</visualize>
             <update_rate>${update_rate}</update_rate>
             <camera>
                 <camera_info_topic>camera/right_camera/camera_info</camera_info_topic>
-                <horizontal_fov>1.089</horizontal_fov>
+                <horizontal_fov>${fov}</horizontal_fov>
                 <image>
                     <format>R8G8B8</format>
@@ -112,6 +147,6 @@
                 </image>
                 <clip>
-                    <near>0.05</near>
-                    <far>8.0</far>
+                    <near>${clip_near}</near>
+                    <far>${clip_far}</far>
                 </clip>
             </camera>

Commit message: Remove redundant description properties

File: description/robot.urdf.xacro (robot description, xacro)
@@ -5,7 +5,7 @@
     <xacro:arg name="camera_name" default="zedm" />
     <xacro:arg name="camera_model" default="zedm" />
-    <xacro:arg name="camera_resolution" default="HD720" />
+    <!-- <xacro:arg name="camera_resolution" default="HD720" /> -->
     <xacro:arg name="use_lidar" default="false" />
-    <xacro:arg name="lidar_update_rate" default="30" />
+    <!-- <xacro:arg name="lidar_update_rate" default="30" /> -->
     <!-- Includes -->
     <xacro:include filename="robot_core.xacro"/>
@@ -17,8 +17,10 @@
     <!-- Build robot model -->
     <xacro:robot_description prefix="$(arg prefix)" camera_name="$(arg camera_name)" camera_model="$(arg camera_model)"/>
+    <!-- lidar_update_rate="$(arg lidar_update_rate)" -->
     <xacro:if value="$(arg use_lidar)">
-        <xacro:lidar_description prefix="$(arg prefix)" lidar_update_rate="$(arg lidar_update_rate)"/>
+        <xacro:lidar_description prefix="$(arg prefix)"/>
     </xacro:if>
     <xacro:vectornav_imu_description prefix="$(arg prefix)"/>
-    <xacro:zed_camera_description prefix="$(arg prefix)" camera_name="$(arg camera_name)" camera_model="$(arg camera_model)" resolution="$(arg camera_resolution)"/>
+    <xacro:zed_camera_description prefix="$(arg prefix)" camera_name="$(arg camera_name)" camera_model="$(arg camera_model)"/>
+    <!-- resolution="$(arg camera_resolution) -->
 </robot>

File: description/zed_camera.xacro (robot description, xacro)
@@ -8,5 +8,6 @@
 <robot xmlns:xacro="http://www.ros.org/wiki/xacro" >
     <!-- Define a macro with a prefix param for the Zed M camera description -->
-    <xacro:macro name="zed_camera_description" params="prefix camera_name=zedm camera_model=zedm resolution=VGA">
+    <xacro:macro name="zed_camera_description" params="prefix camera_name=zedm camera_model=zedm">
+        <!-- resolution=VGA -->
         <!-- Arguments for zed_wrapper/zed_camera -->
         <xacro:arg name="custom_baseline"  default="0.0" />
