Commit message: Fix LiDAR tf

File: description/lidar.xacro (robot description, xacro)
@@ -6,10 +6,10 @@
         <parent link="base_link"/>
         <child link="laser_frame"/>
-        <origin xyz="0.122 0 0.212" rpy="0 0 0"/>
+        <origin xyz="0 0 0.18" rpy="0 0 0"/>
     </joint>
     <!-- LiDAR Link -->
     <link name="laser_frame">
         <visual>
-            <origin xyz="-0.12 0 -0.05"/>
+            <origin xyz="0 0 -0.03"/>
             <geometry>
                 <!-- <cylinder radius="0.08" length="0.04"/> -->
@@ -19,7 +19,7 @@
         </visual>
         <visual>
-            <origin xyz="-0.12 0 -0.09"/>
+            <origin xyz="0 0 -0.04"/>
             <geometry>
-                <cylinder radius="0.02" length="0.09"/>
+                <cylinder radius="0.02" length="0.13"/>
             </geometry>
             <material name="yellow"/>

Commit message: Add lidar update rate arg

File: description/lidar.xacro (robot description, xacro)
@@ -1,75 +1,79 @@
 <?xml version="1.0"?>
 <robot xmlns:xacro="http://www.ros.org/wiki/xacro" >
-    <xacro:property name="PI" value="3.1415926535897931" />
-    <!-- LiDAR Joint -->
-    <joint name="laser_joint" type="fixed">
-        <parent link="base_link"/>
-        <child link="laser_frame"/>
-        <origin xyz="0.122 0 0.212" rpy="0 0 0"/>
-    </joint>
-    <!-- LiDAR Link -->
-    <link name="laser_frame">
-        <visual>
-            <origin xyz="-0.12 0 -0.05"/>
-            <geometry>
-                <!-- <cylinder radius="0.08" length="0.04"/> -->
-                <mesh filename="file://$(find arcs_cohort_description)/meshes/vlp-16.stl"/>
-            </geometry>
-            <material name="yellow"/>
-        </visual>
-        <visual>
-            <origin xyz="-0.12 0 -0.09"/>
-            <geometry>
-                <cylinder radius="0.02" length="0.09"/>
-            </geometry>
-            <material name="yellow"/>
-        </visual>
-        <collision>
-            <geometry>
-                <cylinder radius="0.02" length="0.09"/>
-            </geometry>
-        </collision>
-        <inertial>
-            <origin xyz="0 0 0" rpy="0 0 0"/>
-            <mass value="0.1"/>
-            <inertia ixx="0.0000758333" ixy="0.0" ixz="0.0" iyy="0.0000758333" iyz="0.0" izz="0.000125"/>
-        </inertial>
-    </link>
-    <!-- LiDAR Gazebo -->
-    <gazebo reference="laser_frame">
-        <!-- <material>Gazebo/Black</material> -->
-        <sensor name="laser" type="gpu_lidar">
-            <pose> 0 0 0 0 0 0 </pose>
-            <visualize>false</visualize>
-            <update_rate>30</update_rate>
-            <topic>scan</topic>
-            <gz_frame_id>laser_frame</gz_frame_id>
-            <lidar>
-                <scan>
-                    <horizontal>
-                        <samples>1875</samples>
-                        <resolution>1</resolution>
-                        <min_angle>-${PI}</min_angle>
-                        <max_angle>${PI}</max_angle>
-                    </horizontal>
-                    <vertical>
-                        <samples>16</samples>
-                        <resolution>1</resolution>
-                        <min_angle>-${15.0*PI/180.0}</min_angle>
-                        <max_angle>${15.0*PI/180.0}</max_angle>
-                    </vertical>
-                </scan>
-                <range>
-                    <min>0.3</min>
-                    <max>131.0</max>
-                    <resolution>0.001</resolution>
-                </range>
-                <noise>
-                    <type>gaussian</type>
-                    <mean>0.0</mean>
-                    <stddev>0.0</stddev>
-                </noise>
-            </lidar>
-        </sensor>
-    </gazebo>
+    <!-- Define a lidar description macro -->
+    <xacro:macro name="lidar_description" params="prefix update_rate=30">
+        <!-- Properties -->
+        <xacro:property name="PI" value="3.1415926535897931" />
+        <!-- LiDAR Joint -->
+        <joint name="laser_joint" type="fixed">
+            <parent link="base_link"/>
+            <child link="laser_frame"/>
+            <origin xyz="0.122 0 0.212" rpy="0 0 0"/>
+        </joint>
+        <!-- LiDAR Link -->
+        <link name="laser_frame">
+            <visual>
+                <origin xyz="-0.12 0 -0.05"/>
+                <geometry>
+                    <!-- <cylinder radius="0.08" length="0.04"/> -->
+                    <mesh filename="file://$(find arcs_cohort_description)/meshes/vlp-16.stl"/>
+                </geometry>
+                <material name="yellow"/>
+            </visual>
+            <visual>
+                <origin xyz="-0.12 0 -0.09"/>
+                <geometry>
+                    <cylinder radius="0.02" length="0.09"/>
+                </geometry>
+                <material name="yellow"/>
+            </visual>
+            <collision>
+                <geometry>
+                    <cylinder radius="0.02" length="0.09"/>
+                </geometry>
+            </collision>
+            <inertial>
+                <origin xyz="0 0 0" rpy="0 0 0"/>
+                <mass value="0.1"/>
+                <inertia ixx="0.0000758333" ixy="0.0" ixz="0.0" iyy="0.0000758333" iyz="0.0" izz="0.000125"/>
+            </inertial>
+        </link>
+        <!-- LiDAR Gazebo -->
+        <gazebo reference="laser_frame">
+            <!-- <material>Gazebo/Black</material> -->
+            <sensor name="laser" type="gpu_lidar">
+                <pose> 0 0 0 0 0 0 </pose>
+                <visualize>false</visualize>
+                <update_rate>$(arg update_rate)</update_rate>
+                <topic>scan</topic>
+                <gz_frame_id>laser_frame</gz_frame_id>
+                <lidar>
+                    <scan>
+                        <horizontal>
+                            <samples>1875</samples>
+                            <resolution>1</resolution>
+                            <min_angle>-${PI}</min_angle>
+                            <max_angle>${PI}</max_angle>
+                        </horizontal>
+                        <vertical>
+                            <samples>16</samples>
+                            <resolution>1</resolution>
+                            <min_angle>-${15.0*PI/180.0}</min_angle>
+                            <max_angle>${15.0*PI/180.0}</max_angle>
+                        </vertical>
+                    </scan>
+                    <range>
+                        <min>0.3</min>
+                        <max>131.0</max>
+                        <resolution>0.001</resolution>
+                    </range>
+                    <noise>
+                        <type>gaussian</type>
+                        <mean>0.0</mean>
+                        <stddev>0.0</stddev>
+                    </noise>
+                </lidar>
+            </sensor>
+        </gazebo>
+    </xacro:macro>
 </robot>

Commit message: Update arg names

File: description/lidar.xacro (robot description, xacro)
@@ -2,5 +2,5 @@
 <robot xmlns:xacro="http://www.ros.org/wiki/xacro" >
     <!-- Define a lidar description macro -->
-    <xacro:macro name="lidar_description" params="prefix update_rate=30">
+    <xacro:macro name="lidar_description" params="prefix lidar_update_rate=30">
         <!-- Properties -->
         <xacro:property name="PI" value="3.1415926535897931" />
@@ -45,5 +45,5 @@
                 <pose> 0 0 0 0 0 0 </pose>
                 <visualize>false</visualize>
-                <update_rate>$(arg update_rate)</update_rate>
+                <update_rate>$(arg lidar_update_rate)</update_rate>
                 <topic>scan</topic>
                 <gz_frame_id>laser_frame</gz_frame_id>

File: description/robot.urdf.xacro (robot description, xacro)
@@ -17,5 +17,5 @@
     <xacro:robot_description prefix="$(arg prefix)" camera_name="$(arg camera_name)" camera_model="$(arg camera_model)"/>
     <xacro:if value="$(arg use_lidar)">
-        <xacro:lidar_description prefix="$(arg prefix)" update_rate="$(arg lidar_update_rate)"/>
+        <xacro:lidar_description prefix="$(arg prefix)" lidar_update_rate="$(arg lidar_update_rate)"/>
     </xacro:if>
     <xacro:vectornav_imu_description prefix="$(arg prefix)"/>

Commit message: Refactor prefix handling in robot model

File: description/lidar.xacro (robot description, xacro)
@@ -1,16 +1,22 @@
 <?xml version="1.0"?>
 <robot xmlns:xacro="http://www.ros.org/wiki/xacro" >
-    <!-- Properties -->
-    <xacro:property name="PI" value="3.1415926535897931" />
     <!-- Define a lidar description macro -->
     <xacro:macro name="lidar_description" params="prefix lidar_update_rate=30">
+        <!-- Properties -->
+        <xacro:if value="${prefix != ''}">
+            <xacro:property name="prefix_" value="${prefix}_"/>
+        </xacro:if>
+        <xacro:if value="${prefix == ''}">
+            <xacro:property name="prefix_" value=""/>
+        </xacro:if>
+        <xacro:property name="PI" value="3.1415926535897931" />
         <!-- LiDAR Joint -->
-        <joint name="laser_joint" type="fixed">
-            <parent link="base_link"/>
-            <child link="laser_frame"/>
+        <joint name="${prefix_}laser_joint" type="fixed">
+            <parent link="${prefix_}base_link"/>
+            <child link="${prefix_}laser_frame"/>
             <origin xyz="0 0 0.18" rpy="0 0 0"/>
         </joint>
         <!-- LiDAR Link -->
-        <link name="laser_frame">
+        <link name="${prefix_}laser_frame">
             <visual>
                 <origin xyz="0 0 -0.03"/>
@@ -40,5 +46,5 @@
         </link>
         <!-- LiDAR Gazebo -->
-        <gazebo reference="laser_frame">
+        <gazebo reference="${prefix_}laser_frame">
             <!-- <material>Gazebo/Black</material> -->
             <sensor name="laser" type="gpu_lidar">
@@ -47,5 +53,5 @@
                 <update_rate>$(arg lidar_update_rate)</update_rate>
                 <topic>lidar/scan</topic>
-                <gz_frame_id>laser_frame</gz_frame_id>
+                <gz_frame_id>${prefix_}laser_frame</gz_frame_id>
                 <lidar>
                     <scan>

File: description/robot_core.xacro (robot description, xacro)
@@ -1,7 +1,13 @@
 <?xml version="1.0"?>
 <robot xmlns:xacro="http://www.ros.org/wiki/xacro">
-  <!-- Define a macro with a prefix param for the robot description -->
+  <!-- Define a macro for the robot description -->
   <xacro:macro name="robot_description" params="prefix camera_name=zedm camera_model=zedm">
     <!-- Properties -->
+    <xacro:if value="${prefix != ''}">
+      <xacro:property name="prefix_" value="${prefix}_"/>
+    </xacro:if>
+    <xacro:if value="${prefix == ''}">
+      <xacro:property name="prefix_" value=""/>
+    </xacro:if>
     <xacro:property name="wheel_radius" value="0.08" />
     <xacro:property name="base_footprint_z_offset" value="0.0295" />
@@ -19,5 +25,5 @@
       <color rgba="1 0 0 1"/>
     </material>
-    <link name="${prefix}base_link">
+    <link name="${prefix_}base_link">
       <inertial>
         <origin
@@ -56,11 +62,11 @@
     </link>
     <!-- Robot Footprint -->
-    <link name="${prefix}base_footprint"/>
-    <joint name="${prefix}base_joint" type="fixed">
-      <parent link="${prefix}base_link"/>
-      <child link="${prefix}base_footprint"/>
+    <link name="${prefix_}base_footprint"/>
+    <joint name="${prefix_}base_joint" type="fixed">
+      <parent link="${prefix_}base_link"/>
+      <child link="${prefix_}base_footprint"/>
       <origin xyz="0.0 0.0 -${wheel_radius + base_footprint_z_offset}" rpy="0 0 0"/>
     </joint>
-    <link name="${prefix}front_left_wheel_link">
+    <link name="${prefix_}front_left_wheel_link">
       <inertial>
         <origin
@@ -98,11 +104,11 @@
       </collision>
     </link>
-    <joint name="${prefix}front_left_wheel_joint" type="continuous">
+    <joint name="${prefix_}front_left_wheel_joint" type="continuous">
       <origin xyz="0.12851 0.11738 -0.022625" rpy="-1.5708 0 0" />
-      <parent link="${prefix}base_link" />
-      <child link="${prefix}front_left_wheel_link" />
+      <parent link="${prefix_}base_link" />
+      <child link="${prefix_}front_left_wheel_link" />
       <axis xyz="0 0 1" />
     </joint>
-    <link name="${prefix}front_right_wheel_link">
+    <link name="${prefix_}front_right_wheel_link">
       <inertial>
         <origin
@@ -140,11 +146,11 @@
       </collision>
     </link>
-    <joint name="${prefix}front_right_wheel_joint" type="continuous">
+    <joint name="${prefix_}front_right_wheel_joint" type="continuous">
       <origin xyz="0.12051 -0.11682 -0.022625" rpy="1.5708 0 0" />
-      <parent link="${prefix}base_link" />
-      <child link="${prefix}front_right_wheel_link" />
+      <parent link="${prefix_}base_link" />
+      <child link="${prefix_}front_right_wheel_link" />
       <axis xyz="0 0 -1" />
     </joint>
-    <link name="${prefix}back_left_wheel_link">
+    <link name="${prefix_}back_left_wheel_link">
       <inertial>
         <origin
@@ -182,11 +188,11 @@
       </collision>
     </link>
-    <joint name="${prefix}back_left_wheel_joint" type="continuous">
+    <joint name="${prefix_}back_left_wheel_joint" type="continuous">
       <origin xyz="-0.11949 0.11738 -0.022625" rpy="-1.5708 0 0" />
-      <parent link="${prefix}base_link" />
-      <child link="${prefix}back_left_wheel_link" />
+      <parent link="${prefix_}base_link" />
+      <child link="${prefix_}back_left_wheel_link" />
       <axis xyz="0 0 1" />
     </joint>
-    <link name="${prefix}back_right_wheel_link">
+    <link name="${prefix_}back_right_wheel_link">
       <inertial>
         <origin
@@ -224,11 +230,11 @@
       </collision>
     </link>
-    <joint name="${prefix}back_right_wheel_joint" type="continuous">
+    <joint name="${prefix_}back_right_wheel_joint" type="continuous">
       <origin xyz="-0.12749 -0.11682 -0.022625" rpy="1.5708 0 0" />
-      <parent link="${prefix}base_link" />
-      <child link="${prefix}back_right_wheel_link" />
+      <parent link="${prefix_}base_link" />
+      <child link="${prefix_}back_right_wheel_link" />
       <axis xyz="0 0 -1" />
     </joint>
-    <link name="${prefix}imu_link">
+    <link name="${prefix_}imu_link">
       <inertial>
         <origin
@@ -270,11 +276,11 @@
       </collision>
     </link>
-    <joint name="${prefix}imu_joint" type="fixed">
+    <joint name="${prefix_}imu_joint" type="fixed">
       <origin xyz="0.0022791 0.00028171 0.01489" rpy="0 0 0" />
-      <parent link="${prefix}base_link" />
-      <child link="${prefix}imu_link" />
+      <parent link="${prefix_}base_link" />
+      <child link="${prefix_}imu_link" />
       <axis xyz="0 0 0" />
     </joint>
-    <link name="${prefix}${camera_name}_camera_mount_link">
+    <link name="${prefix_}${camera_name}_camera_mount_link">
       <inertial>
         <origin
@@ -312,8 +318,8 @@
       </collision>
     </link>
-    <joint name="${prefix}camera_mount_joint" type="fixed">
+    <joint name="${prefix_}camera_mount_joint" type="fixed">
       <origin xyz="0.14426 0.00028171 0.094535" rpy="0 0 0" />
-      <parent link="${prefix}base_link" />
-      <child link="${prefix}${camera_name}_camera_mount_link" />
+      <parent link="${prefix_}base_link" />
+      <child link="${prefix_}${camera_name}_camera_mount_link" />
       <axis xyz="0 0 0" />
     </joint>

File: description/vectornav_imu.xacro (robot description, xacro)
@@ -3,5 +3,12 @@
   <!-- Define a macro with a prefix param for the VectorNav IMU description -->
   <xacro:macro name="vectornav_imu_description" params="prefix">
-    <gazebo reference="${prefix}imu_link">
+    <!-- Properties -->
+    <xacro:if value="${prefix != ''}">
+        <xacro:property name="prefix_" value="${prefix}_"/>
+    </xacro:if>
+    <xacro:if value="${prefix == ''}">
+        <xacro:property name="prefix_" value=""/>
+    </xacro:if>
+    <gazebo reference="${prefix_}imu_link">
         <sensor name="vn100_imu" type="imu">
             <always_on>true</always_on>

File: description/zed_camera.xacro (robot description, xacro)
@@ -9,21 +9,16 @@
     <!-- Define a macro with a prefix param for the Zed M camera description -->
     <xacro:macro name="zed_camera_description" params="prefix camera_name=zedm camera_model=zedm resolution=VGA">
-        <!-- Arguments for zed_wrapper/zed_camera -->
-        <xacro:arg name="custom_baseline"  default="0.0" />
-        <xacro:arg name="enable_gnss"   default="false" />
-        <xacro:arg name="gnss_x" default="0.0" />
-        <xacro:arg name="gnss_y" default="0.0" />
-        <xacro:arg name="gnss_z" default="0.0" />
-        <!-- Include zed_wrapper/zed_camera description -->
-        <xacro:include filename="$(find zed_wrapper)/urdf/zed_macro.urdf.xacro" />
-        <xacro:zed_camera name="$(arg camera_name)" model="$(arg camera_model)" custom_baseline="$(arg custom_baseline)" enable_gnss="$(arg enable_gnss)">
-                <origin xyz="$(arg gnss_x) $(arg gnss_y) $(arg gnss_z)" rpy="0 0 0"/>
-        </xacro:zed_camera>
-        <!--Camera-->
-        <joint name="${prefix}${camera_name}_camera_mount_to_camera" type="fixed">
-            <parent link="${prefix}${camera_name}_camera_mount_link"/>
-            <child link="${camera_name}_camera_link"/>
-            <origin xyz="0.037592 -0.0065 -0.02273" rpy="0 ${30*(M_PI/180)} 0" />
-        </joint>
+        <!-- Properties -->
+        <xacro:if value="${prefix != ''}">
+            <xacro:property name="prefix_" value="${prefix}_"/>
+        </xacro:if>
+        <xacro:if value="${prefix == ''}">
+            <xacro:property name="prefix_" value=""/>
+        </xacro:if>
+        <xacro:property name="custom_baseline" value="0.0" />
+        <xacro:property name="enable_gnss" value="false" />
+        <xacro:property name="gnss_x" value="0.0" />
+        <xacro:property name="gnss_y" value="0.0" />
+        <xacro:property name="gnss_z" value="0.0" />
         <xacro:if value="${resolution == 'HD2K'}">
             <xacro:property name="resolution_width" value="2208" />
@@ -80,7 +75,18 @@
             </gazebo>
         </xacro:if>
+        <!-- Include zed_wrapper/zed_camera description -->
+        <xacro:include filename="$(find zed_wrapper)/urdf/zed_macro.urdf.xacro" />
+        <xacro:zed_camera name="$(arg camera_name)" model="$(arg camera_model)" custom_baseline="${custom_baseline}" enable_gnss="${enable_gnss}">
+                <origin xyz="${gnss_x} ${gnss_y} ${gnss_z}" rpy="0 0 0"/>
+        </xacro:zed_camera>
+        <!--Camera-->
+        <joint name="${prefix_}${camera_name}_camera_mount_to_camera" type="fixed">
+            <parent link="${prefix_}${camera_name}_camera_mount_link"/>
+            <child link="${camera_name}_camera_link"/>
+            <origin xyz="0.037592 -0.0065 -0.02273" rpy="0 ${30*(M_PI/180)} 0" />
+        </joint>
         <!-- Left Camera Gazebo -->
         <gazebo reference="${camera_name}_left_camera_frame">
-            <sensor name="${prefix}left_camera" type="rgbd_camera">
+            <sensor name="${prefix_}left_camera" type="rgbd_camera">
                 <topic>camera/left_camera</topic>
                 <gz_frame_id>${camera_name}_left_camera_frame</gz_frame_id>
@@ -105,5 +111,5 @@
         <!-- Right Camera Gazebo -->
         <gazebo reference="${camera_name}_right_camera_frame">
-            <sensor name="${prefix}right_camera" type="camera">
+            <sensor name="${prefix_}right_camera" type="camera">
                 <topic>camera/right_camera/image</topic>
                 <gz_frame_id>${camera_name}_right_camera_frame</gz_frame_id>
