Commit message: Refactor prefix handling

File: description/lidar.xacro (robot description, xacro)
@@ -2,5 +2,5 @@
 <robot xmlns:xacro="http://www.ros.org/wiki/xacro" >
     <!-- Define a lidar description macro -->
-    <xacro:macro name="lidar_description" params="prefix lidar_update_rate=30">
+    <xacro:macro name="lidar_description" params="namespace prefix lidar_update_rate=30">
         <!-- Properties -->
         <xacro:if value="${prefix != ''}">
@@ -52,5 +52,5 @@
                 <visualize>false</visualize>
                 <update_rate>$(arg lidar_update_rate)</update_rate>
-                <topic>lidar/scan</topic>
+                <topic>${namespace}/lidar/scan</topic>
                 <gz_frame_id>${prefix_}laser_frame</gz_frame_id>
                 <lidar>

File: description/robot.urdf.xacro (robot description, xacro)
@@ -2,4 +2,5 @@
 <robot xmlns:xacro="http://www.ros.org/wiki/xacro" name="robot">
     <!-- Arguments -->
+    <xacro:arg name="namespace" default="" />
     <xacro:arg name="prefix" default="" />
     <xacro:arg name="camera_name" default="zedm" />
@@ -27,14 +28,14 @@
     <xacro:robot_description prefix="$(arg prefix)" camera_name="$(arg camera_name)" camera_model="$(arg camera_model)"/>
     <xacro:if value="$(arg use_lidar)">
-        <xacro:lidar_description prefix="$(arg prefix)" lidar_update_rate="$(arg lidar_update_rate)"/>
+        <xacro:lidar_description namespace="$(arg namespace)" prefix="$(arg prefix)" lidar_update_rate="$(arg lidar_update_rate)"/>
     </xacro:if>
-    <xacro:vectornav_imu_description prefix="$(arg prefix)"/>
-    <xacro:zed_camera_description prefix="$(arg prefix)" camera_name="$(arg camera_name)" camera_model="$(arg camera_model)" resolution="$(arg camera_resolution)"/>
+    <xacro:vectornav_imu_description namespace="$(arg namespace)" prefix="$(arg prefix)"/>
+    <xacro:zed_camera_description namespace="$(arg namespace)" prefix="$(arg prefix)" camera_name="$(arg camera_name)" camera_model="$(arg camera_model)" resolution="$(arg camera_resolution)"/>
     <!-- Conditionally call the appropriate Gazebo plugin description -->
     <xacro:if value="$(arg use_ros2_control)">
-        <xacro:gazebo_ros2_control_plugin_description prefix="$(arg prefix)"/>
+        <xacro:gazebo_ros2_control_plugin_description namespace="$(arg namespace)" prefix="$(arg prefix)"/>
     </xacro:if>
     <xacro:unless value="$(arg use_ros2_control)">
-        <xacro:gazebo_diff_drive_plugin_description prefix="$(arg prefix)"/>
+        <xacro:gazebo_diff_drive_plugin_description namespace="$(arg namespace)" prefix="$(arg prefix)"/>
     </xacro:unless>
 </robot>

File: description/vectornav_imu.xacro (robot description, xacro)
@@ -2,5 +2,5 @@
 <robot xmlns:xacro="http://www.ros.org/wiki/xacro" >
   <!-- Define a macro with a prefix param for the VectorNav IMU description -->
-  <xacro:macro name="vectornav_imu_description" params="prefix">
+  <xacro:macro name="vectornav_imu_description" params="namespace prefix">
     <!-- Properties -->
     <xacro:if value="${prefix != ''}">
@@ -14,5 +14,5 @@
             <always_on>true</always_on>
             <update_rate>800</update_rate>
-            <topic>imu</topic>
+            <topic>$(arg namespace)/imu</topic>
             <imu>
                 <angular_velocity>

File: description/zed_camera.xacro (robot description, xacro)
@@ -8,5 +8,5 @@
 <robot xmlns:xacro="http://www.ros.org/wiki/xacro" >
     <!-- Define a macro with a prefix param for the Zed M camera description -->
-    <xacro:macro name="zed_camera_description" params="prefix camera_name=zedm camera_model=zedm resolution=VGA">
+    <xacro:macro name="zed_camera_description" params="namespace prefix camera_name=zedm camera_model=zedm resolution=VGA">
         <!-- Properties -->
         <xacro:if value="${prefix != ''}">
@@ -77,23 +77,23 @@
         <!-- Include zed_wrapper/zed_camera description -->
         <xacro:include filename="$(find zed_wrapper)/urdf/zed_macro.urdf.xacro" />
-        <xacro:zed_camera name="$(arg camera_name)" model="$(arg camera_model)" custom_baseline="${custom_baseline}" enable_gnss="${enable_gnss}">
-                <origin xyz="${gnss_x} ${gnss_y} ${gnss_z}" rpy="0 0 0"/>
+        <xacro:zed_camera name="${prefix_ + camera_name}" model="$(arg camera_model)" custom_baseline="${custom_baseline}" enable_gnss="${enable_gnss}">
+            <origin xyz="${gnss_x} ${gnss_y} ${gnss_z}" rpy="0 0 0"/>
         </xacro:zed_camera>
         <!--Camera-->
-        <joint name="${prefix_}${camera_name}_camera_mount_to_camera" type="fixed">
-            <parent link="${prefix_}${camera_name}_camera_mount_link"/>
-            <child link="${camera_name}_camera_link"/>
+        <joint name="${prefix_ + camera_name}_camera_mount_to_camera" type="fixed">
+            <parent link="${prefix_ + camera_name}_camera_mount_link"/>
+            <child link="${prefix_ + camera_name}_camera_link"/>
             <origin xyz="0.037592 -0.0065 -0.02273" rpy="0 ${30*(M_PI/180)} 0" />
         </joint>
         <!-- Left Camera Gazebo -->
-        <gazebo reference="${camera_name}_left_camera_frame">
+        <gazebo reference="${prefix_ + camera_name}_left_camera_frame">
             <sensor name="${prefix_}left_camera" type="rgbd_camera">
-                <topic>camera/left_camera</topic>
-                <gz_frame_id>${camera_name}_left_camera_frame</gz_frame_id>
+                <topic>${namespace}/camera/left_camera</topic>
+                <gz_frame_id>${prefix_ + camera_name}_left_camera_frame</gz_frame_id>
                 <always_on>1</always_on>
                 <update_rate>${update_rate}</update_rate>
                 <visualize>true</visualize>
                 <camera>
-                    <camera_info_topic>camera/left_camera_info</camera_info_topic>
+                    <camera_info_topic>${namespace}/camera/left_camera_info</camera_info_topic>
                     <horizontal_fov>${fov}</horizontal_fov>
                     <image>
@@ -110,12 +110,12 @@
         </gazebo>
         <!-- Right Camera Gazebo -->
-        <gazebo reference="${camera_name}_right_camera_frame">
+        <gazebo reference="${prefix_ + camera_name}_right_camera_frame">
             <sensor name="${prefix_}right_camera" type="camera">
-                <topic>camera/right_camera/image</topic>
-                <gz_frame_id>${camera_name}_right_camera_frame</gz_frame_id>
+                <topic>${namespace}/camera/right_camera/image</topic>
+                <gz_frame_id>${prefix_ + camera_name}_right_camera_frame</gz_frame_id>
                 <visualize>true</visualize>
                 <update_rate>${update_rate}</update_rate>
                 <camera>
-                    <camera_info_topic>camera/right_camera/camera_info</camera_info_topic>
+                    <camera_info_topic>${namespace}/camera/right_camera/camera_info</camera_info_topic>
                     <horizontal_fov>${fov}</horizontal_fov>
                     <image>

Commit message: Remove gazebo references from description files

File: description/lidar.xacro (robot description, xacro)
@@ -6,5 +6,5 @@
     <xacro:macro name="lidar_description" params="prefix lidar_update_rate=30">
         <!-- LiDAR Joint -->
-        <joint name="laser_joint" type="fixed">
+        <joint name="${prefix}laser_joint" type="fixed">
             <parent link="base_link"/>
             <child link="laser_frame"/>
@@ -12,5 +12,5 @@
         </joint>
         <!-- LiDAR Link -->
-        <link name="laser_frame">
+        <link name="${prefix}laser_frame">
             <visual>
                 <origin xyz="0 0 -0.03"/>
@@ -39,41 +39,4 @@
             </inertial>
         </link>
-        <!-- LiDAR Gazebo -->
-        <gazebo reference="laser_frame">
-            <!-- <material>Gazebo/Black</material> -->
-            <sensor name="laser" type="gpu_lidar">
-                <pose> 0 0 0 0 0 0 </pose>
-                <visualize>false</visualize>
-                <update_rate>$(arg lidar_update_rate)</update_rate>
-                <topic>lidar/scan</topic>
-                <gz_frame_id>laser_frame</gz_frame_id>
-                <lidar>
-                    <scan>
-                        <horizontal>
-                            <samples>1875</samples>
-                            <resolution>1</resolution>
-                            <min_angle>-${PI}</min_angle>
-                            <max_angle>${PI}</max_angle>
-                        </horizontal>
-                        <vertical>
-                            <samples>16</samples>
-                            <resolution>1</resolution>
-                            <min_angle>-${15.0*PI/180.0}</min_angle>
-                            <max_angle>${15.0*PI/180.0}</max_angle>
-                        </vertical>
-                    </scan>
-                    <range>
-                        <min>0.3</min>
-                        <max>131.0</max>
-                        <resolution>0.001</resolution>
-                    </range>
-                    <noise>
-                        <type>gaussian</type>
-                        <mean>0.0</mean>
-                        <stddev>0.0</stddev>
-                    </noise>
-                </lidar>
-            </sensor>
-        </gazebo>
     </xacro:macro>
 </robot>

File: description/robot.urdf.xacro (robot description, xacro)
@@ -8,8 +8,6 @@
     <xacro:arg name="use_lidar" default="false" />
     <xacro:arg name="lidar_update_rate" default="30" />
-    <xacro:arg name="use_ros2_control" default="false" />
     <!-- Includes -->
     <xacro:include filename="robot_core.xacro"/>
-    <xacro:include filename="lidar.xacro"/>
     <xacro:include filename="vectornav_imu.xacro"/>
     <xacro:include filename="zed_camera.xacro"/>
@@ -17,11 +15,4 @@
         <xacro:include filename="lidar.xacro"/>
     </xacro:if>
-    <!-- Include Gazebo plugins -->
-    <xacro:if value="$(arg use_ros2_control)">
-        <xacro:include filename="$(find arcs_cohort_gazebo_sim)/control/gazebo_ros2_control_plugin.xacro"/>
-    </xacro:if>
-    <xacro:unless value="$(arg use_ros2_control)">
-        <xacro:include filename="$(find arcs_cohort_gazebo_sim)/control/gazebo_diff_drive_plugin.xacro"/>
-    </xacro:unless>
     <!-- Build robot model -->
     <xacro:robot_description prefix="$(arg prefix)" camera_name="$(arg camera_name)" camera_model="$(arg camera_model)"/>
@@ -31,10 +22,3 @@
     <xacro:vectornav_imu_description prefix="$(arg prefix)"/>
     <xacro:zed_camera_description prefix="$(arg prefix)" camera_name="$(arg camera_name)" camera_model="$(arg camera_model)" resolution="$(arg camera_resolution)"/>
-    <!-- Conditionally call the appropriate Gazebo plugin description -->
-    <xacro:if value="$(arg use_ros2_control)">
-        <xacro:gazebo_ros2_control_plugin_description prefix="$(arg prefix)"/>
-    </xacro:if>
-    <xacro:unless value="$(arg use_ros2_control)">
-        <xacro:gazebo_diff_drive_plugin_description prefix="$(arg prefix)"/>
-    </xacro:unless>
 </robot>

File: description/robot_core.xacro (robot description, xacro)
@@ -230,50 +230,4 @@
       <axis xyz="0 0 -1" />
     </joint>
-    <link name="${prefix}imu_link">
-      <inertial>
-        <origin
-          xyz="-0.000894812057582933 9.60259274576658E-06 -0.00456943294796108"
-          rpy="0 0 0" />
-        <mass
-          value="0.0065760792742103" />
-        <inertia
-          ixx="3.78511408547619E-07"
-          ixy="4.67820105640642E-11"
-          ixz="1.00912927862616E-08"
-          iyy="3.79926110271894E-07"
-          iyz="-5.01543493566598E-12"
-          izz="7.19032056380139E-07" />
-      </inertial>
-      <visual>
-        <origin
-          xyz="0 0 0"
-          rpy="0 0 0" />
-        <geometry>
-          <mesh
-            filename="file://$(find arcs_cohort_description)/meshes/new_imu.stl" />
-        </geometry>
-        <material
-          name="">
-          <color
-            rgba="0.792156862745098 0.819607843137255 0.933333333333333 1" />
-        </material>
-      </visual>
-      <collision>
-        <origin
-          xyz="0 0 0"
-          rpy="0 0 0" />
-        <geometry>
-          <mesh
-            filename="file://$(find arcs_cohort_description)/meshes/new_imu.stl" />
-          <!-- <box size = "0.03 0.025 0.01"/> -->
-        </geometry>
-      </collision>
-    </link>
-    <joint name="${prefix}imu_joint" type="fixed">
-      <origin xyz="0.0022791 0.00028171 0.01489" rpy="0 0 0" />
-      <parent link="${prefix}base_link" />
-      <child link="${prefix}imu_link" />
-      <axis xyz="0 0 0" />
-    </joint>
     <link name="${prefix}${camera_name}_camera_mount_link">
       <inertial>

File: description/vectornav_imu.xacro (robot description, xacro)
@@ -3,53 +3,50 @@
   <!-- Define a macro with a prefix param for the VectorNav IMU description -->
   <xacro:macro name="vectornav_imu_description" params="prefix">
-    <gazebo reference="${prefix}imu_link">
-        <sensor name="vn100_imu" type="imu">
-            <always_on>true</always_on>
-            <update_rate>800</update_rate>
-            <topic>imu</topic>
-            <imu>
-                <angular_velocity>
-                    <x>
-                    <noise type="gaussian">
-                        <mean>0.0</mean>
-                        <stddev>2e-4</stddev>
-                    </noise>
-                    </x>
-                    <y>
-                    <noise type="gaussian">
-                        <mean>0.0</mean>
-                        <stddev>2e-4</stddev>
-                    </noise>
-                    </y>
-                    <z>
-                    <noise type="gaussian">
-                        <mean>0.0</mean>
-                        <stddev>2e-4</stddev>
-                    </noise>
-                    </z>
-                </angular_velocity>
-                <linear_acceleration>
-                    <x>
-                    <noise type="gaussian">
-                        <mean>0.0</mean>
-                        <stddev>1.7e-2</stddev>
-                    </noise>
-                    </x>
-                    <y>
-                    <noise type="gaussian">
-                        <mean>0.0</mean>
-                        <stddev>1.7e-2</stddev>
-                    </noise>
-                    </y>
-                    <z>
-                    <noise type="gaussian">
-                        <mean>0.0</mean>
-                        <stddev>1.7e-2</stddev>
-                    </noise>
-                    </z>
-                </linear_acceleration>
-            </imu>
-        </sensor>
-    </gazebo>
+    <link name="${prefix}imu_link">
+        <inertial>
+            <origin
+                xyz="-0.000894812057582933 9.60259274576658E-06 -0.00456943294796108"
+                rpy="0 0 0" />
+            <mass
+                value="0.0065760792742103" />
+            <inertia
+                ixx="3.78511408547619E-07"
+                ixy="4.67820105640642E-11"
+                ixz="1.00912927862616E-08"
+                iyy="3.79926110271894E-07"
+                iyz="-5.01543493566598E-12"
+                izz="7.19032056380139E-07" />
+        </inertial>
+        <visual>
+            <origin
+                xyz="0 0 0"
+                rpy="0 0 0" />
+            <geometry>
+                <mesh
+                filename="file://$(find arcs_cohort_description)/meshes/new_imu.stl" />
+            </geometry>
+            <material
+                name="">
+                <color
+                rgba="0.792156862745098 0.819607843137255 0.933333333333333 1" />
+            </material>
+        </visual>
+        <collision>
+            <origin
+                xyz="0 0 0"
+                rpy="0 0 0" />
+            <geometry>
+                <mesh
+                filename="file://$(find arcs_cohort_description)/meshes/new_imu.stl" />
+                <!-- <box size = "0.03 0.025 0.01"/> -->
+            </geometry>
+        </collision>
+    </link>
+    <joint name="${prefix}imu_joint" type="fixed">
+        <origin xyz="0.0022791 0.00028171 0.01489" rpy="0 0 0" />
+        <parent link="${prefix}base_link" />
+        <child link="${prefix}imu_link" />
+        <axis xyz="0 0 0" />
+    </joint>
   </xacro:macro>
 </robot>

File: description/zed_camera.xacro (robot description, xacro)
@@ -26,103 +26,4 @@
             <origin xyz="0.037592 -0.0065 -0.02273" rpy="0 ${30*(M_PI/180)} 0" />
         </joint>
-        <xacro:if value="${resolution == 'HD2K'}">
-            <xacro:property name="resolution_width" value="2208" />
-            <xacro:property name="resolution_height" value="1242" />
-            <xacro:property name="update_rate" value="15" />
-        </xacro:if>
-        <xacro:if value="${resolution == 'HD1080'}">
-            <xacro:property name="resolution_width" value="1920" />
-            <xacro:property name="resolution_height" value="1080" />
-            <xacro:property name="update_rate" value="30" />
-        </xacro:if>
-        <xacro:if value="${resolution == 'HD720'}">
-            <xacro:property name="resolution_width" value="1280" />
-            <xacro:property name="resolution_height" value="720" />
-            <xacro:property name="update_rate" value="60" />
-        </xacro:if>
-        <xacro:if value="${resolution == 'VGA'}">
-            <xacro:property name="resolution_width" value="672" />
-            <xacro:property name="resolution_height" value="376" />
-            <xacro:property name="update_rate" value="100" />
-        </xacro:if>
-        <xacro:if value="${camera_model == 'zed'}">
-            <xacro:property name="baseline" value="0.12" />
-            <xacro:property name="fov" value="2.0" />
-            <xacro:property name="clip_near" value="0.3" />
-            <xacro:property name="clip_far" value="25" />
-            <!-- Gazebo color -->
-            <gazebo reference="${camera_model}_camera_center">
-                <material>Gazebo/Grey</material>
-            </gazebo>
-        </xacro:if>
-        <xacro:if value="${camera_model == 'zedm'}">
-            <xacro:property name="baseline" value="0.06" />
-            <xacro:property name="fov" value="2.0" />
-            <xacro:property name="clip_near" value="0.1" />
-            <xacro:property name="clip_far" value="15" />
-            <!-- Add IMU for ZED -->
-            <!-- <xacro:imu_gazebo name="${camera_name}" frame="${camera_name}_imu_frame_gazebo" /> -->
-            <!-- Gazebo color -->
-            <gazebo reference="${camera_model}_camera_center">
-                <material>Gazebo/DarkGrey</material>
-            </gazebo>
-        </xacro:if>
-        <xacro:if value="${camera_model == 'zed2'}">
-            <xacro:property name="baseline" value="0.12" />
-            <xacro:property name="fov" value="1.8" />
-            <xacro:property name="clip_near" value="0.2" />
-            <xacro:property name="clip_far" value="20" />
-            <!-- Add IMU for ZED -->
-            <xacro:imu_gazebo name="${camera_name}" frame="${camera_name}_imu_frame_gazebo" />
-            <!-- Gazebo color -->
-            <gazebo reference="${camera_model}_camera_center">
-                <material>Gazebo/Black</material>
-            </gazebo>
-        </xacro:if>
-        <!-- Left Camera Gazebo -->
-        <gazebo reference="${camera_name}_left_camera_frame">
-            <sensor name="${prefix}left_camera" type="rgbd_camera">
-                <topic>camera/left_camera</topic>
-                <gz_frame_id>${camera_name}_left_camera_frame</gz_frame_id>
-                <always_on>1</always_on>
-                <update_rate>${update_rate}</update_rate>
-                <visualize>true</visualize>
-                <camera>
-                    <camera_info_topic>camera/left_camera_info</camera_info_topic>
-                    <horizontal_fov>${fov}</horizontal_fov>
-                    <image>
-                        <format>R8G8B8</format>
-                        <width>${resolution_width}</width>
-                        <height>${resolution_height}</height>
-                    </image>
-                    <clip>
-                        <near>${clip_near}</near>
-                        <far>${clip_far}</far>
-                    </clip>
-                </camera>
-            </sensor>
-        </gazebo>
-        <!-- Right Camera Gazebo -->
-        <gazebo reference="${camera_name}_right_camera_frame">
-            <sensor name="${prefix}right_camera" type="camera">
-                <topic>camera/right_camera/image</topic>
-                <gz_frame_id>${camera_name}_right_camera_frame</gz_frame_id>
-                <visualize>true</visualize>
-                <update_rate>${update_rate}</update_rate>
-                <camera>
-                    <camera_info_topic>camera/right_camera/camera_info</camera_info_topic>
-                    <horizontal_fov>${fov}</horizontal_fov>
-                    <image>
-                        <format>R8G8B8</format>
-                        <width>${resolution_width}</width>
-                        <height>${resolution_height}</height>
-                    </image>
-                    <clip>
-                        <near>${clip_near}</near>
-                        <far>${clip_far}</far>
-                    </clip>
-                </camera>
-            </sensor>
-        </gazebo>
     </xacro:macro>
 </robot>

Commit message: Remove comments

File: description/lidar.xacro (robot description, xacro)
@@ -4,5 +4,5 @@
     <xacro:property name="PI" value="3.1415926535897931" />
     <!-- Define a lidar description macro -->
-    <xacro:macro name="lidar_description" params="prefix lidar_update_rate=30">
+    <xacro:macro name="lidar_description" params="prefix">
         <!-- LiDAR Joint -->
         <joint name="${prefix}laser_joint" type="fixed">

File: description/robot.urdf.xacro (robot description, xacro)
@@ -5,7 +5,5 @@
     <xacro:arg name="camera_name" default="zedm" />
     <xacro:arg name="camera_model" default="zedm" />
-    <!-- <xacro:arg name="camera_resolution" default="HD720" /> -->
     <xacro:arg name="use_lidar" default="false" />
-    <!-- <xacro:arg name="lidar_update_rate" default="30" /> -->
     <!-- Includes -->
     <xacro:include filename="robot_core.xacro"/>
@@ -17,5 +15,4 @@
     <!-- Build robot model -->
     <xacro:robot_description prefix="$(arg prefix)" camera_name="$(arg camera_name)" camera_model="$(arg camera_model)"/>
-    <!-- lidar_update_rate="$(arg lidar_update_rate)" -->
     <xacro:if value="$(arg use_lidar)">
         <xacro:lidar_description prefix="$(arg prefix)"/>
@@ -23,4 +20,3 @@
     <xacro:vectornav_imu_description prefix="$(arg prefix)"/>
     <xacro:zed_camera_description prefix="$(arg prefix)" camera_name="$(arg camera_name)" camera_model="$(arg camera_model)"/>
-    <!-- resolution="$(arg camera_resolution) -->
 </robot>
